File: Cluster.kicad_sch (KiCad schematic)
At the start: 73 parts, among them J1 DTM06-2S nickel, 12V input (s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, J2 SWD Tag-Connect, J3 Panox BH021WVC02 - center spe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, Q1 PMV37ENEA automotive (AEC-Q10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, Q2 PMV37ENEA automotive (AEC-Q10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, Q3 PMV37ENEA automotive (AEC-Q10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, U1 NXP S32K144 automotive (AEC-Q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, U10 TPS7A16-Q1 (AEC-Q100 G1), U11 Bridgetek BT817AQ automotive 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, U2 LMR33630-Q1 (AEC-Q100 G1), U3 LM74700-Q1 (AEC-Q100 G1), U4 TLV733P-Q1 (AEC-Q100 G1), U5 NXP TJA1043T automotive CAN t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, U6 Raystar RFA401280B-AYW-DNF1 -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, U7 Raystar RFA401280B-AYW-DNF1 -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, U8 Raystar RFA401280B-AYW-DNF1 -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, U9 Raystar RFA401280B-AYW-DNF1 -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, Y1 8MHz (AEC-Q200), Y2 12MHz (AEC-Q200)

Commit message: Step 6: CAN0 + sensor harness connector; schematic complete
J7 (real Molex KK-254 5-position, same family thermo-pcb already
established) lands CAN0_H/CAN0_L and the 3 resistive-sender taps.
Battery voltage needs no separate harness pin - it already reads
VIN_PROT, the same tap the power connector provides.

This closes out every step of the original build-out plan. Updated
README.md, this file's own header docstring, and its on-sheet NOTES to
reflect the finished state: ERC-clean at the same 4 baseline findings
every sibling board's completed schematic carries, no guessed pins or
values anywhere. PCB layout/routing/DRC/BOM are the next, not-yet-
started phase.

Co-Authored-By: Claude Sonnet 5 <noreply@anthropic.com>
Parts:
- added J7: DTM06-5S nickel, CAN0 + 3x sender input (sealed), Connector_Molex:Molex_KK-254_AE-6410-05A_1x05_P2.54mm_Vertical, symbol Cluster:CONN_HARNESS
Connections:
- net ADC_FUEL: now also J7.3 (FUEL_SENSE)
- net ADC_OIL: now also J7.4 (OIL_SENSE)
- net ADC_TEMP: now also J7.5 (TEMP_SENSE)
- net CAN0_H: now also J7.1 (CAN0_H)
- net CAN0_L: now also J7.2 (CAN0_L)
Other:
- note added: "(ERC can't trace power through a ferrite/FET/diode); J2 SWCLK pin_not_driven"
- note added: "(genuinely driven off-sheet by the debug probe). PCB layout/routing/DRC/BOM are"
- note added: "+ R12/R13 generate it. RGB666 wiring follows the module's own documented bit"
- note added: "3. U1 (S32K144) pin numbers are REAL - fixed pins verified against NXP's Reference"
- note added: "4. U5 (TJA1043T) reused verbatim from ecu-pcb's own real CAN transceiver circuit."
- note added: "6. J1 (power) and J7 (CAN0 + 3x sender) both land real Molex KK-254/Phoenix MKDS"
- note added: "7. Schematic is FULLY WIRED (all 6 plan steps done, 2026-09-22). kicad-cli sch erc"
- note added: "Manual (same research thermo-pcb/manifold-pcb did for this part/package);"
- note added: "Manual's own embedded IO-signal-table attachment, cross-checked pin-by-pin for"
- note added: "U10/U11/J3 (BT817AQ + ST7701S speedo): BT817A's VCC1V2 core rail is a genuine"
- note added: "U6-U9 (GC9A01) use Raystar's real RFA401280B-AYW-DNF1 pinout - backlight is a"
- note added: "bare LED pair (not a logic pin), driven from +5V with a shared MOSFET switch."
- note added: "board-side connectors, sealed DTM06 nickel pigtails on the outboard end - same"
- note added: "collisions programmatically, not by eye. No generic placeholders anywhere."
- note added: "external 1.28V supply (not internally regulated) - U10 (TPS7A16-Q1, adjustable)"
- note added: "for a dash-mounted (not engine-bay) board."
- note added: "from the sender's own real resistance curve (README.md), not a shared guess."
- note added: "order (DB0=Blue LSB..DB17=Red MSB). R16-R20 (sensor dividers) are each sized"
- note added: "peripheral pins (LPSPI1/LPSPI2/FlexCAN0/4xADC/GPIO) verified against the same"
- note added: "real strategy thermo-pcb established. Not yet re-confirmed as the right choice"
- note added: "separate, not-yet-started next phases."
- note added: "shows exactly 4 findings, all the same expected tool-limitation pattern every"
- note added: "sibling board's FINISHED schematic carries: VDDA/U2-VIN/+5V power_pin_not_driven"
- note removed: "2x12-bit ADC x16ch=32 channels - the ~26 real pins Cluster's aux-gauge SPI bus +"
- note removed: "3. U1 pin numbers are REAL, verified against NXP's S32K1xx Reference Manual (same"
- note removed: "4. Real S32K144 pin/peripheral budget (README.md, verified 2026-09-22 against NXP's"
- note removed: "6. J1 (power landing) reuses thermo-pcb's real Phoenix MKDS + outboard DTM06-2S"
- note removed: "64-pin package leaves after the fixed pins wired here - NOT yet pin-mux"
- note removed: "7. kicad-cli sch erc is expected to show only the same tool-limitation findings"
- note removed: "BT817AQ QSPI + CAN0 + 4x ADC will need fit comfortably inside the ~58 GPIO this"
- note removed: "SWCLK pin_not_driven - genuinely driven off-sheet by the debug probe)."
- note removed: "every sibling board's schematic has at this stage (VDDA/U2-VIN/+5V"
- note removed: "for a dash-mounted (not engine-bay) board; flagged for the connector pass."
- note removed: "generic placeholders. ONLY fixed pins (crystal/SWD/RESET/power) are wired this"
- note removed: "own S32K1xx Data Sheet Rev.15): this part has 3x LPSPI, 3x FlexCAN (1 w/ FD),"
- note removed: "pass - see this file's own header docstring for what's deliberately deferred."
- note removed: "pigtail strategy as a starting point - not yet re-confirmed as the right choice"
- note removed: "power_pin_not_driven - ERC can't trace power through a ferrite/FET/diode; J2"
- note removed: "research thermo-pcb/manifold-pcb already did for this exact part/package) - not"
- note removed: "researched pin-by-pin, that's the next real work before those subsystems wire."
