File: Cluster.kicad_pcb (KiCad board)
At the start: 4 copper layers, 447.1 x 102.5 mm, 74 parts, among them J1 DTM06-2S nickel, 12V input (s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, J2 SWD Tag-Connect, J3 Panox BH021WVC02 - center spe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, J7 DTM06-5S nickel, CAN0 + 3x se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, Q1 PMV37ENEA automotive (AEC-Q10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, Q2 PMV37ENEA automotive (AEC-Q10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, Q3 PMV37ENEA automotive (AEC-Q10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, U1 NXP S32K144 automotive (AEC-Q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, U10 TPS7A16-Q1 (AEC-Q100 G1), U11 Bridgetek BT817AQ automotive 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, U2 LMR33630-Q1 (AEC-Q100 G1), U3 LM74700-Q1 (AEC-Q100 G1), U4 TLV733P-Q1 (AEC-Q100 G1), U5 NXP TJA1043T automotive CAN t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, U6 Raystar RFA401280B-AYW-DNF1 -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, U7 Raystar RFA401280B-AYW-DNF1 -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, U8 Raystar RFA401280B-AYW-DNF1 -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, U9 Raystar RFA401280B-AYW-DNF1 -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, Y1 8MHz (AEC-Q200), Y2 12MHz (AEC-Q200)

Commit message: Spread PCB placement into real functional zones + back-silk logo
User feedback: the first-pass layout bunched everything into one
corner, leaving most of the board empty. Reworked into real zones -
each display gets its own local cluster of immediate support parts
directly above it (the speedo's whole BT817AQ+LDO+crystal subsystem
included, a real short-trace reason not just visual balance), and the
board-wide subsystems (power, MCU, CAN0, backlight switch, sender
dividers) pack independently then arrange left-to-right with equal
spacing across the board's real full width - same "bucket into
functional blocks" precedent ecu-pcb's own PCB already established.

Also added the real back-silkscreen "Jessie's Cars" logo every sibling
board carries, sized generously (up to 80mm) for Cluster's own wide,
mostly-empty back side.

Still 447.1x102.5mm, still DRC-clean except the same benign
lib_footprint_mismatch category every sibling board's finished PCB has.

Co-Authored-By: Claude Sonnet 5 <noreply@anthropic.com>
Parts:
- moved C17 324.6 mm to (105.1, 246.8)
- moved C3 297.5 mm to (185.5, 164.5)
- moved C1 287.6 mm to (175.6, 164.5)
- moved C11 272.7 mm to (175.6, 167.9)
- moved R6 253.5 mm to (100.1, 246.8)
- moved R3 252.9 mm to (190.5, 167.9)
- moved J7 226.5 mm to (323.2, 167.2)
- moved C20 222.4 mm to (480.4, 246.8)
- moved C12 213.2 mm to (180.6, 167.9)
- moved C27 189.8 mm to (315.4, 241.6)
- moved C21 188.4 mm to (300.6, 238.1)
- moved C5 185.4 mm to (267.8, 164.5)
- moved Q2 178.2 mm to (410.4, 165.4)
- moved R9 177.5 mm to (475.5, 246.8)
- moved C2 173.5 mm to (180.6, 164.5)
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
Commit message: Replace back-silkscreen logo with an original tach-face design
User asked for something cooler than the reused sibling-board logo.
Drew a real tachometer face (0-8 sweep, redline arc, resting needle,
"x1000 RPM" caption) plus a CLUSTER wordmark directly as KiCad graphic
primitives (GrCircle/GrArc/GrLine/GrText) - original artwork, not
traced from any existing source, genuinely on-theme for an instrument
cluster board.

Real detail that needed getting right: back-layer shapes aren't
auto-mirrored by KiCad the way text glyphs are (which use an effects
flag instead) - every primitive routes through one shared mirror
helper so the constructive layout code stays in natural left-to-right
reading order. One real DRC hit along the way (bold 13mm CLUSTER text
wider than expected, overlapping the gauge face) fixed with real
spacing margin, confirmed by an actual render, not just clearing DRC.

Co-Authored-By: Claude Sonnet 5 <noreply@anthropic.com>
Other:
- board text added: "0"
- board text added: "1"
- board text added: "2"
- board text added: "3"
- board text added: "4"
- board text added: "5"
- board text added: "6"
- board text added: "7"
- board text added: "8"
- board text added: "CLUSTER"
- board text added: "DIGITAL INSTRUMENT CLUSTER"
- board text added: "JESSIE'S CARS"
- board text added: "x1000 RPM"
