File: Cluster.kicad_pcb (KiCad board)
At the start: 4 copper layers, 447.1 x 102.5 mm, 74 parts, among them J1 DTM06-2S nickel, 12V input (s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, J2 SWD Tag-Connect, J3 Panox BH021WVC02 - center spe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, J7 DTM06-5S nickel, CAN0 + 3x se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, Q1 PMV37ENEA automotive (AEC-Q10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, Q2 PMV37ENEA automotive (AEC-Q10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, Q3 PMV37ENEA automotive (AEC-Q10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, U1 NXP S32K144 automotive (AEC-Q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, U10 TPS7A16-Q1 (AEC-Q100 G1), U11 Bridgetek BT817AQ automotive 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, U2 LMR33630-Q1 (AEC-Q100 G1), U3 LM74700-Q1 (AEC-Q100 G1), U4 TLV733P-Q1 (AEC-Q100 G1), U5 NXP TJA1043T automotive CAN t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, U6 Raystar RFA401280B-AYW-DNF1 -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, U7 Raystar RFA401280B-AYW-DNF1 -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, U8 Raystar RFA401280B-AYW-DNF1 -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, U9 Raystar RFA401280B-AYW-DNF1 -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, Y1 8MHz (AEC-Q200), Y2 12MHz (AEC-Q200)

Commit message: Right-size board height to real content, not the opening's own max
User feedback: "i think we can make it smaller. no reason to make it so
big right?" - correct. The board's width genuinely can't shrink below
~441mm (the 5 connectors have to reach across the real dash-opening
width to land under their own gauge holes), but the height had no such
constraint - it was anchored to the opening's own 105.5mm inner
dimension as if the board needed to fill it vertically, which was
never actually required.

Reworked the layout order: pack local clusters and core zones first to
find their real sizes, then derive board_height from what's actually
stacked (margins + display row + local clusters + core zones) instead
of anchoring to the oversized opening dimension.

Board: 447.1x102.5mm -> 447.1x51.3mm, under half the height, same
width, still DRC-clean (same accepted-exception categories as before).

Co-Authored-By: Claude Sonnet 5 <noreply@anthropic.com>
Parts:
- moved C17 28.6 mm to (105.1, 218.2)
- moved C18 28.6 mm to (200.8, 218.2)
- moved C19 28.6 mm to (392.2, 218.2)
- moved C20 28.6 mm to (480.4, 218.2)
- moved C21 28.6 mm to (300.6, 209.5)
- moved C22 28.6 mm to (305.5, 209.5)
- moved C23 28.6 mm to (320.4, 209.5)
- moved C24 28.6 mm to (300.6, 212.9)
- moved C25 28.6 mm to (305.5, 212.9)
- moved C26 28.6 mm to (310.5, 212.9)
- moved C27 28.6 mm to (315.4, 212.9)
- moved C31 28.6 mm to (495.3, 218.2)
- moved J3 28.6 mm to (294.0, 226.9)
- moved Q3 28.6 mm to (295.1, 210.4)
- moved R12 28.6 mm to (310.5, 209.5)
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Other:
- board size 447.1 x 102.5 mm -> 447.1 x 51.3 mm

Commit message: Add 6 real M3 standoff holes; fix two bugs this surfaced
4 corners + 2 along the top edge - a board this long and thin needs
more than 2 support points to avoid real flex/vibration in a
dash-mounted automotive environment.

Two real bugs caught and fixed by the same build/verify/fix loop:
1. A first attempt placed the 2 extra holes at naive 1/3 and 2/3
   board-width fractions and landed on R4/R5 and U1 - fixed by using
   the actual empty gaps between core zones (captured while they're
   being placed) instead of a guessed fraction.
2. Adding the holes shrank the tach-face artwork's own safe drawing
   area (GAUGE_R 21.5mm -> 15.6mm), but its internal tick/number/
   caption geometry was all fixed mm offsets tuned for the original
   size - produced 27 real overlapping-silkscreen DRC hits. Fixed by
   scaling every internal offset and text size proportionally to the
   actual radius.

Still DRC-clean (same accepted-exception categories), board unchanged
at 447.1x51.3mm.

Co-Authored-By: Claude Sonnet 5 <noreply@anthropic.com>
Parts:
- added MH1: MountingHole_3.2mm_M3, MountingHole:MountingHole_3.2mm_M3, F.Cu at (80.5, 191.3)
- added MH2: MountingHole_3.2mm_M3, MountingHole:MountingHole_3.2mm_M3, F.Cu at (513.5, 191.3)
- added MH3: MountingHole_3.2mm_M3, MountingHole:MountingHole_3.2mm_M3, F.Cu at (80.5, 228.7)
- added MH4: MountingHole_3.2mm_M3, MountingHole:MountingHole_3.2mm_M3, F.Cu at (513.5, 228.7)
- added MH5: MountingHole_3.2mm_M3, MountingHole:MountingHole_3.2mm_M3, F.Cu at (208.1, 191.3)
- added MH6: MountingHole_3.2mm_M3, MountingHole:MountingHole_3.2mm_M3, F.Cu at (438.4, 191.3)

Commit message: Route the PCB: 251/252 nets via FreeRouting, VIN_PROT trunk widened, GND/+3V3 zones poured
route_board.py adapts thermo-pcb's own DSN/SES FreeRouting pipeline
(export via pcbnew.ExportSpecctraDSN, headless FreeRouting, import via
pcbnew.ImportSpecctraSES, then two additive post-route passes: widen
the VIN_PROT power trunk from its 0.2mm routing width back up to
0.6mm, then pour+fill GND/+3V3 zones on the inner layers, one zone per
subprocess to dodge a known pcbnew multi-zone-fill segfault).

FreeRouting converged 251/252 nets on the first pass; one net
(AUX_DC3, U9 pin 13 -> U1 pin 24) stayed stuck across 6 retries - real
autorouter congestion around this board's 0.5mm-pitch parts, needs a
short hand-route in pcbnew before the board is real. DRC is otherwise
clean: same documented silk/footprint categories as the unrouted
board, nothing new introduced by routing.

Also fixes a real bug found while verifying the routed result: the
board's paper size was never actually set on the kiutils Board object
(build_pcb.py computed offsets assuming A2 but kiutils silently kept
its own A4 default), so the drawn page frame didn't match where the
board's content actually sat. One-line fix (board.paper.paperSize =
"A2"); board was regenerated and re-routed from scratch rather than
hand-patched, landing the same 251/252 result.

Co-Authored-By: Claude Sonnet 5 <noreply@anthropic.com>
Routing:
- net GND: track 0.00 -> 810.4 mm, vias 0 -> 25
- net +3V3: track 0.00 -> 661.2 mm, vias 0 -> 17
- net +5V: track 0.00 -> 478.1 mm, vias 0 -> 11
- net AUX_VLED_RTN: track 0.00 -> 431.0 mm, vias 0 -> 5
- net AUX_RST: track 0.00 -> 426.6 mm, vias 0 -> 6
- net LPSPI2_SCK: track 0.00 -> 421.7 mm, vias 0 -> 5
- net LPSPI2_SOUT: track 0.00 -> 414.4 mm, vias 0 -> 5
- net VIN_PROT: track 0.00 -> 397.8 mm, vias 0 -> 6
- net ADC_BATT: track 0.00 -> 273.9 mm, vias 0 -> 3
- net AUX_CS3: track 0.00 -> 271.2 mm, vias 0 -> 3
- net ADC_TEMP: track 0.00 -> 255.3 mm, vias 0 -> 2
- net ADC_OIL: track 0.00 -> 247.4 mm, vias 0 -> 3
- net ADC_FUEL: track 0.00 -> 244.0 mm, vias 0 -> 2
- net LPSPI2_SIN: track 0.00 -> 194.9 mm, vias 0 -> 3
- net BL_EN: track 0.00 -> 181.1 mm, vias 0 -> 3
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- added copper zone on In2.Cu, net +3V3
- added copper zone on In1.Cu, net GND

Commit message: Fully route the PCB: 252/252 nets, 0 unrouted
The prior commit landed 251/252 (one net, AUX_DC3, stuck across 6
FreeRouting retries). FreeRouting is stochastic and its outcome tracks
the exact DSN content, so regenerating the board fresh (no code
change) and re-routing gave the export a different implicit seed -
this cycle converged fully, 0 unrouted, in 7 auto-router passes.
DRC-clean, same documented categories as before, no hand-routing
needed.

Co-Authored-By: Claude Sonnet 5 <noreply@anthropic.com>
Routing:
- net AUX_DC3: track 0.00 -> 270.5 mm, vias 0 -> 3
- net +3V3: track 661.2 -> 718.5 mm, vias 17 -> 18
- net GND: track 810.4 -> 769.0 mm, vias 25 -> 24
- net +5V: track 478.1 -> 454.8 mm, vias 11 -> 12
- net VIN_PROT: track 397.8 -> 377.9 mm, vias 6 -> 10
- net AUX_CS1: track 55.9 -> 37.5 mm
- net LPSPI2_SCK: track 421.7 -> 434.7 mm
- net AUX_RST: track 426.6 -> 414.8 mm
- net SPD_G3: track 39.3 -> 29.2 mm
- net AUX_DC0: track 145.2 -> 135.2 mm, vias 2 -> 3
- net LPSPI1_SIN: track 58.9 -> 49.9 mm
- net AUX_VLED_RTN: track 431.0 -> 422.9 mm
- net VIN_FUSED: track 92.6 -> 84.7 mm, vias 3 -> 4
- net SPD_G6: track 31.6 -> 39.1 mm
- net LPSPI2_SOUT: track 414.4 -> 421.4 mm
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