File: gauges/ClusterGauges.kicad_pcb (KiCad board)
At the start: 4 copper layers, 447.1 x 42.6 mm, 64 parts, among them J1 DTM06-2S nickel, 12V input (s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, J2 SWD Tag-Connect, J7 DTM06-5S nickel, CAN0 + 3x se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, Q1 PMV37ENEA automotive (AEC-Q10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, Q2 PMV37ENEA automotive (AEC-Q10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, U1 NXP S32K144 automotive (AEC-Q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, U2 LMR33630-Q1 (AEC-Q100 G1), U3 LM74700-Q1 (AEC-Q100 G1), U4 TLV733P-Q1 (AEC-Q100 G1), U5 NXP TJA1043T automotive CAN t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, U6 Raystar RFA401280B-AYW-DNF1 -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, U7 Raystar RFA401280B-AYW-DNF1 -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, U8 Raystar RFA401280B-AYW-DNF1 -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, U9 Raystar RFA401280B-AYW-DNF1 -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, Y1 8MHz (AEC-Q200)

Commit message: gauges: route board and generate real BOM
Routed ClusterGauges.kicad_pcb with FreeRouting (0 unrouted on the
first attempt) plus post-route GND/+3V3 zone pours and VIN_PROT trunk
widening, adapted from the top-level cluster-pcb/route_board.py.

Found and fixed a real bug in the process: widen_trunks()'s
TRACK_CLEARANCE was set to 0.15mm to match the netclass "clearance"
field, but kicad-cli's actual enforced DRC minimum is 0.2mm (every
.kicad_pro in this family leaves design_settings.rules.min_clearance
unset, so KiCad falls back to its own stock default regardless of the
netclass value). A first route+widen+zone pass produced 235 real
clearance violations, all on widened VIN_PROT segments. Fixed the
constant, regenerated the board fresh, re-routed - 0 unrouted, DRC
clean except the same benign lib_footprint_mismatch/silk categories
every sibling board's finished PCB carries.

Added build_bom.py, adapted from ecu-pcb's own real, generated-not-
hand-maintained BOM generator: real MPNs for every non-passive that
build_schematic.py's own comments cite, parametric passives, a real
fuse element/holder split, and real harness pigtail connectors (DTM06-
2S/5S) as separate non-placement lines. 58/58 real parts covered.

Co-Authored-By: Claude Sonnet 5 <noreply@anthropic.com>
Routing:
- net GND: track 0.00 -> 672.6 mm, vias 0 -> 23
- net +3V3: track 0.00 -> 551.6 mm, vias 0 -> 16
- net +5V: track 0.00 -> 482.1 mm, vias 0 -> 8
- net AUX_VLED_RTN: track 0.00 -> 437.9 mm, vias 0 -> 5
- net AUX_RST: track 0.00 -> 425.6 mm, vias 0 -> 5
- net LPSPI2_SOUT: track 0.00 -> 424.2 mm, vias 0 -> 5
- net LPSPI2_SCK: track 0.00 -> 422.1 mm, vias 0 -> 6
- net VIN_PROT: track 0.00 -> 392.1 mm, vias 0 -> 6
- net ADC_BATT: track 0.00 -> 289.8 mm, vias 0 -> 2
- net AUX_CS3: track 0.00 -> 275.0 mm, vias 0 -> 4
- net AUX_DC3: track 0.00 -> 270.6 mm, vias 0 -> 3
- net ADC_TEMP: track 0.00 -> 257.4 mm, vias 0 -> 2
- net ADC_OIL: track 0.00 -> 249.8 mm, vias 0 -> 3
- net ADC_FUEL: track 0.00 -> 246.0 mm, vias 0 -> 3
- net LPSPI2_SIN: track 0.00 -> 195.3 mm, vias 0 -> 3
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- added copper zone on In2.Cu, net +3V3
- added copper zone on In1.Cu, net GND

Commit message: gauges rev B: private CAN1 link, Hall speed input, ignition input
Gateway architecture: this board is the only car-bus node and aggregates for
display/. Adds a second TCAN1044V-Q1 (CAN1, pins 51/52 from NXP's own IO
table), a 12V Hall pulse input into FTM1_CH4 (pin 58), and an ignition input
(J1 pin 3 to GPIO pin 59, pin-interrupt wake per the RM's AWIC table). Both
inputs are clamped with BAV99-Q. ERC baseline unchanged (4), routed 0
unconnected, BOM regenerated.

Co-Authored-By: Claude Sonnet 5.5 <noreply@anthropic.com>
Parts:
- added C40: 100nF VCC decouple (AEC-Q200), Capacitor_SMD:C_0603_1608Metric, F.Cu at (347.2, 194.4)
- added C41: 100nF VIO decouple (AEC-Q200), Capacitor_SMD:C_0603_1608Metric, F.Cu at (352.2, 194.4)
- added C42: 4.7nF SPLIT stabilization (AEC-Q200), Capacitor_SMD:C_0603_1608Metric, F.Cu at (357.1, 194.4)
- added C43: 1nF input filter (AEC-Q200), Capacitor_SMD:C_0603_1608Metric, F.Cu at (421.9, 194.4)
- added C44: 10nF input filter (AEC-Q200), Capacitor_SMD:C_0603_1608Metric, F.Cu at (436.8, 194.4)
- added D10: BAV99-Q input clamp (AEC-Q101), Package_TO_SOT_SMD:SOT-23, F.Cu at (395.8, 195.4)
- added D11: BAV99-Q input clamp (AEC-Q101), Package_TO_SOT_SMD:SOT-23, F.Cu at (401.7, 195.4)
- added J8: KK-254 22-27-2031, private link to display/ J3 (DTM06-3S pi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, Connector_Molex:Molex_KK-254_AE-6410-03A_1x03_P2.54mm_Vertical, F.Cu at (327.5, 197.1)
- added J9: KK-254 22-27-2021, Hall speed sender (signal + ground), Connector_Molex:Molex_KK-254_AE-6410-02A_1x02_P2.54mm_Vertical, F.Cu at (388.5, 198.0)
- added R40: 10k STB pulldown, normal mode while MCU resets (AEC-Q200), Resistor_SMD:R_0603_1608Metric, F.Cu at (362.1, 194.4)
- added R41: 60R split termination (AEC-Q200), Resistor_SMD:R_0603_1608Metric, F.Cu at (367.1, 194.4)
- added R42: 60R split termination (AEC-Q200), Resistor_SMD:R_0603_1608Metric, F.Cu at (372.0, 194.4)
- added R43: 4.7k pull-up to VIN_PROT for open-collector senders (AEC-Q2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, Resistor_SMD:R_0603_1608Metric, F.Cu at (407.1, 194.4)
- added R44: 33k series (AEC-Q200), Resistor_SMD:R_0603_1608Metric, F.Cu at (412.0, 194.4)
- added R45: 15k divider bottom (AEC-Q200), Resistor_SMD:R_0603_1608Metric, F.Cu at (417.0, 194.4)
- added R46: 56k series (AEC-Q200), Resistor_SMD:R_0603_1608Metric, F.Cu at (426.9, 194.4)
- added R47: 27k divider bottom (AEC-Q200), Resistor_SMD:R_0603_1608Metric, F.Cu at (431.9, 194.4)
- added U10: TCAN1044V-Q1 (AEC-Q100 G1), Package_SO:SOIC-8_3.9x4.9mm_P1.27mm, F.Cu at (340.1, 196.5)
- J1: value DTM06-2S nickel, 12V input (sealed) -> DTM06-3S nickel, 12V input + ignition (sealed); footprint TerminalBlock_Phoenix:TerminalBlock_Phoenix_MKDS-1,5-2-5.08_1x02_P5.08mm_Horizontal -> TerminalBlock_Phoenix:TerminalBlock_Phoenix_MKDS-1,5-3-5.08_1x03_P5.08mm_Horizontal
- moved C14 62.0 mm to (292.8, 194.4)
- moved C13 62.0 mm to (287.9, 194.4)
- moved C15 62.0 mm to (297.8, 194.4)
- moved C16 62.0 mm to (302.8, 194.4)
- moved J7 62.0 mm to (261.2, 197.1)
- moved R4 62.0 mm to (307.7, 194.4)
- moved R5 62.0 mm to (312.7, 194.4)
- moved U5 62.0 mm to (279.8, 197.4)
- moved MH6 59.1 mm to (379.3, 195.7)
- moved R2 50.2 mm to (135.3, 199.6)
- moved Q2 41.4 mm to (451.8, 195.4)
- moved R10 41.4 mm to (457.2, 194.4)
- moved R11 41.4 mm to (462.2, 194.4)
- moved C8 41.3 mm to (241.4, 194.4)
- moved C6 41.3 mm to (231.5, 194.4)
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Connections:
- U1 pad 51: (no net) -> CAN1_TX
- U1 pad 52: (no net) -> CAN1_RX
- U1 pad 58: (no net) -> SPEED_IN
- U1 pad 59: (no net) -> IGN_SENSE
- U1 pad 60: (no net) -> CAN1_STB
Routing:
- net IGN_RAW: track 0.00 -> 314.5 mm, vias 0 -> 1
- net IGN_SENSE: track 0.00 -> 255.6 mm, vias 0 -> 3
- net SPEED_IN: track 0.00 -> 242.3 mm, vias 0 -> 2
- net CAN1_STB: track 0.00 -> 178.2 mm, vias 0 -> 3
- net CAN1_TX: track 0.00 -> 149.8 mm, vias 0 -> 2
- net CAN1_RX: track 0.00 -> 148.6 mm, vias 0 -> 2
- net BL_EN: track 181.4 -> 273.2 mm
- net LPSPI2_SIN: track 195.3 -> 276.7 mm
- net GND: track 672.6 -> 739.3 mm, vias 23 -> 25
- net ADC_OIL: track 249.8 -> 315.8 mm
- net ADC_FUEL: track 246.0 -> 309.5 mm
- net ADC_TEMP: track 257.4 -> 315.8 mm
- net +3V3: track 551.6 -> 602.8 mm, vias 16 -> 20
- net CAN1_L: track 0.00 -> 50.3 mm, vias 0 -> 2
- net AUX_CS0: track 142.4 -> 95.3 mm, vias 3 -> 2
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
Commit message: Prepare both boards for fabrication: real power-stage values, orderable BOMs, fab packages
display/ power stage was placeholders inherited from fascia-pcb (RILIM, OV top,
RT, FB top...). Values are now calculated from the LM74930-Q1, LM61460-Q1 and
TLV767-Q1 datasheets, with real packages (1u XEL5030 inductor, 1206 caps, 2 mohm
sense resistor, polymer bulk cap). gauges/ buck inductor (XAL5050, Isat above the
LMR33630 current limit) and input/output capacitors fixed per its datasheet.
tools/passive_catalog.py maps every passive to a real MPN (entries flagged
verified or pattern). fab/build_fab.py writes gerbers, drill, CPL and BOM CSVs
and refuses boards with unconnected nets. Silkscreen text raised to the fab
minimum; gauges input zones moved beside the MCU. Both boards re-routed, 0
unconnected.

Co-Authored-By: Claude Sonnet 5.5 <noreply@anthropic.com>
Parts:
- added C45: 22uF 10V X7R COUT (AEC-Q200), Capacitor_SMD:C_1206_3216Metric, F.Cu at (144.7, 200.4)
- added C46: 220nF 50V CHF at VIN (AEC-Q200), Capacitor_SMD:C_0603_1608Metric, F.Cu at (160.4, 203.3)
- C1: value 10uF X7R (AEC-Q200) -> 10uF 50V X7R CIN (AEC-Q200); footprint Capacitor_SMD:C_0603_1608Metric -> Capacitor_SMD:C_1210_3225Metric
- C2: value 22uF X7R (AEC-Q200) -> 22uF 10V X7R COUT (AEC-Q200); footprint Capacitor_SMD:C_0603_1608Metric -> Capacitor_SMD:C_1206_3216Metric
- L1: value 10uH power (AEC-Q200) -> 10uH power XAL5050-103ME (AEC-Q200); footprint Inductor_SMD:L_1210_3225Metric -> Inductor_SMD:L_Coilcraft_XAL5050-XXX
- L2: footprint Inductor_SMD:L_1210_3225Metric -> Inductor_SMD:L_0603_1608Metric
- moved D10 127.3 mm to (268.5, 195.4)
- moved D11 127.3 mm to (274.3, 195.4)
- moved J9 127.3 mm to (261.1, 198.0)
- moved R45 127.3 mm to (289.6, 194.4)
- moved R46 127.3 mm to (299.6, 194.4)
- moved R47 127.3 mm to (304.5, 194.4)
- moved C43 127.3 mm to (294.6, 194.4)
- moved C44 127.3 mm to (309.5, 194.4)
- moved R43 127.3 mm to (279.7, 194.4)
- moved R44 127.3 mm to (284.7, 194.4)
- moved C14 123.1 mm to (416.0, 194.4)
- moved C13 123.1 mm to (411.0, 194.4)
- moved C15 123.1 mm to (420.9, 194.4)
- moved C16 123.1 mm to (425.9, 194.4)
- moved J7 123.1 mm to (384.3, 197.1)
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Routing:
- net CAN0_TX: track 95.6 -> 221.4 mm
- net IGN_SENSE: track 255.6 -> 130.4 mm, vias 3 -> 2
- net CAN0_RX: track 97.9 -> 222.2 mm
- net SPEED_IN: track 242.3 -> 118.7 mm
- net CAN0_EN: track 104.6 -> 223.3 mm, vias 3 -> 2
- net CAN0_STB_N: track 104.8 -> 220.3 mm
- net IGN_RAW: track 314.5 -> 208.7 mm
- net +3V3: track 602.8 -> 551.0 mm, vias 20 -> 19
- net GND: track 739.3 -> 694.2 mm, vias 25 -> 28
- net VIN_FUSED: track 86.7 -> 56.0 mm, vias 2 -> 1
- net +5V: track 472.3 -> 497.6 mm, vias 11 -> 12
- net VIN_PROT: track 416.7 -> 439.5 mm, vias 10 -> 9
- net VCAP: track 22.5 -> 7.83 mm
- net SW: track 41.2 -> 26.8 mm, vias 3 -> 2
- net VCC_INT: track 28.7 -> 16.0 mm
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
Commit message: Fix review findings: MOSFET pinout, gauges surge front end, converter cells, DSI
Review of 2026-10-03 found real defects; fixes and measured results:
- Nexperia PMV55ENEA/PMV37ENEA pinout is G=1, S=2, D=3: display Q1-Q3 and
  gauges Q2 had source/drain swapped. Fixed in both schematics.
- gauges/ now has the same LM74930-Q1 surge-protected front end as display/
  (5 mohm sense, OV clamp), a 5 A/32 V blade fuse on display/ (the MF-RG500 PTC
  was a 16 V part), and sender inputs with series resistor, clamp and filter.
- Converters are placed as cells around their ICs (tools/cellplace.py).
  display: SW_5V 55.6 -> 11.6 mm, boost/inverter/backlight SW 75 -> 7-13 mm,
  LM61460 input caps 57 -> 4.7-7.5 mm. gauges: SW 26.8 -> 8.7 mm, input caps 4.5 mm.
- display DSI pairs are planned by dsi_route.py after the autorouter: legs
  10.6-11.2 mm, at most 0.6 mm skew in a pair (was 64-85 mm, 21 mm skew).
- In1 is a GND plane for the router on display/ (about 925 mm of slow signals
  still cross it, down from 2615); forbidding signals there left 6-122
  connections unrouted. gauges/ keeps the old flow (planes claimed there made
  the real GND zone split into islands).
- display: USB (J13) and console UART (J12) bring-up headers, SoM and socket
  split into separate BOM lines, README rewritten.
- gauges: orderable MCU part number, DNP parts get their own BOM line and are
  left out of the placement file, 5 mohm sense resistor in the catalog.

Both boards: 0 unconnected, independent kicad-cli DRC with only accepted
categories; fab packages rebuilt. Nothing is fabricated or tested.

Co-Authored-By: Claude Sonnet 5.5 <noreply@anthropic.com>
Parts:
- removed C10: 100nF charge-pump cap (AEC-Q200), Capacitor_SMD:C_0603_1608Metric
- added C47: 100nF CVS (50V), Capacitor_SMD:C_0603_1608Metric, F.Cu at (135.0, 197.7)
- added C48: 100nF CCAP (50V), Capacitor_SMD:C_0603_1608Metric, F.Cu at (124.2, 198.1)
- added C49: 100nF CTMR, Capacitor_SMD:C_0603_1608Metric, F.Cu at (135.0, 194.3)
- added D12: BAV99-Q fuel input clamp (AEC-Q101), Package_TO_SOT_SMD:SOT-23, F.Cu at (448.4, 188.8)
- added D13: BAV99-Q oil input clamp (AEC-Q101), Package_TO_SOT_SMD:SOT-23, F.Cu at (454.2, 188.8)
- added D14: BAV99-Q temp input clamp (AEC-Q101), Package_TO_SOT_SMD:SOT-23, F.Cu at (460.1, 188.8)
- added D15: BAV99-Q battery divider clamp (AEC-Q101), Package_TO_SOT_SMD:SOT-23, F.Cu at (478.5, 219.5)
- added Q3: PMV55ENEA pass (HGATE), Package_TO_SOT_SMD:SOT-23, F.Cu at (129.5, 188.8)
- added R48: 49.9R 1% RSET, Resistor_SMD:R_0603_1608Metric, F.Cu at (124.2, 191.3)
- added R49: 5m 1% sense (Susumu KRL3216E-M-R005-F-T5), Resistor_SMD:R_1206_3216Metric, F.Cu at (124.6, 194.7)
- added R50: 80.6k 1% RILIM (1.5A breaker), Resistor_SMD:R_0603_1608Metric, F.Cu at (135.0, 190.9)
- added R51: 100k OV top, Resistor_SMD:R_0603_1608Metric, F.Cu at (132.6, 200.3)
- added R52: 2.05k OV bot (clamp 29.9V), Resistor_SMD:R_0603_1608Metric, F.Cu at (132.6, 202.2)
- added R53: 100k UV top, Resistor_SMD:R_0603_1608Metric, F.Cu at (136.0, 200.3)
- added R54: 11.5k UV bot (cut-off 5.5V), Resistor_SMD:R_0603_1608Metric, F.Cu at (136.0, 202.2)
- added R55: 1k fuel ADC series (AEC-Q200), Resistor_SMD:R_0603_1608Metric, F.Cu at (495.2, 187.8)
- added R56: 1k oil ADC series (AEC-Q200), Resistor_SMD:R_0603_1608Metric, F.Cu at (500.2, 187.8)
- added R57: 1k temp ADC series (AEC-Q200), Resistor_SMD:R_0603_1608Metric, F.Cu at (465.5, 191.3)
- D1: value SMCJ33A automotive (AEC-Q101) -> SMCJ33A automotive (AEC-Q101) on the fused input, ahead of the LM74930
- Q1: value PMV37ENEA automotive (AEC-Q101) -> PMV55ENEA ideal diode (DGATE)
- R16: value 47R fuel pull-up, self-calculated for the sender's 10-73R range (AEC-Q200) -> 1k fuel pull-up to +3V3 (11mW at a 10R sender) (AEC-Q200)
- R17: value 47R oil pressure pull-up, self-calculated for the sender's 10-70R range (AEC-Q200) -> 1k oil pull-up to +3V3 (AEC-Q200)
- R18: value 100R coolant temp pull-up, self-calculated for the sender's 10-300R range (AEC-Q200) -> 1k coolant temp pull-up to +3V3 (AEC-Q200)
- U3: value LM74700-Q1 (AEC-Q100 G1) -> LM74930-Q1 (AEC-Q100 G1); footprint Package_TO_SOT_SMD:SOT-23-6 -> Package_DFN_QFN:Texas_RGE0024H_VQFN-24-1EP_4x4mm_P0.5mm_EP2.7x2.7mm
- moved C2 81.3 mm to (87.5, 208.9), turned to -90 degrees
- moved C1 66.6 mm to (102.4, 204.6), turned to 90 degrees
- moved C46 63.6 mm to (96.9, 200.9)
- moved C11 59.3 mm to (96.9, 209.2), turned to 180 degrees
- moved C45 57.3 mm to (87.5, 203.9), turned to 90 degrees
- moved R1 56.6 mm to (187.8, 191.3)
- moved C3 54.2 mm to (107.5, 201.1), turned to 180 degrees
- moved U2 47.4 mm to (97.9, 205.1), turned to 0 degrees
- moved L1 46.1 mm to (92.0, 205.3), turned to 180 degrees
- moved U4 44.1 mm to (112.5, 202.2), turned to 90 degrees
- moved C12 36.1 mm to (100.3, 209.2)
- moved Q1 33.6 mm to (129.0, 201.3), turned to -90 degrees
- moved C43 33.0 mm to (262.3, 187.8)
- moved C44 33.0 mm to (277.2, 187.8)
- moved R43 33.0 mm to (247.4, 187.8)
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Connections:
- D1 pad 1: VIN_PROT -> VIN_FUSED
- J7 pad 3: ADC_FUEL -> SENDER_FUEL
- J7 pad 4: ADC_OIL -> SENDER_OIL
- J7 pad 5: ADC_TEMP -> SENDER_TEMP
- Q1 pad 1: GATE_DRV -> DGATE
- Q1 pad 2: VIN_FUSED -> COMMON
- Q2 pad 2: AUX_VLED_RTN -> GND
- Q2 pad 3: GND -> AUX_VLED_RTN
- R16 pad 2: ADC_FUEL -> SENDER_FUEL
- R17 pad 2: ADC_OIL -> SENDER_OIL
- R18 pad 2: ADC_TEMP -> SENDER_TEMP
- U3 pad 1: VCAP -> DGATE
- U3 pad 2: GND -> COMMON
- U3 pad 3: VIN_FUSED -> SW_SENSE
- U3 pad 4: VIN_PROT -> UVLO_DIV
- U3 pad 5: GATE_DRV -> OV_DIV
Routing:
- net SENDER_OIL: track 0.00 -> 142.5 mm, vias 0 -> 2
- net SENDER_FUEL: track 0.00 -> 139.0 mm, vias 0 -> 3
- net SENDER_TEMP: track 0.00 -> 119.8 mm, vias 0 -> 2
- net GND: track 694.2 -> 810.8 mm, vias 28 -> 23
- net +3V3: track 551.0 -> 620.5 mm, vias 19 -> 18
- net IGN_RAW: track 208.7 -> 154.7 mm
- net ADC_BATT: track 319.1 -> 356.5 mm, vias 3 -> 2
- net AUX_CS1: track 27.5 -> 63.2 mm
- net VIN_PROT: track 439.5 -> 474.5 mm, vias 9 -> 8
- net RESET: track 70.0 -> 35.9 mm
- net AUX_DC1: track 19.2 -> 51.8 mm
- net AUX_CS3: track 316.3 -> 348.4 mm
- net ADC_FUEL: track 310.7 -> 342.7 mm, vias 3 -> 4
- net AUX_DC2: track 214.8 -> 246.7 mm
- net AUX_DC3: track 312.1 -> 344.1 mm
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Other:
- board size 447.1 x 42.6 mm -> 447.1 x 55.8 mm
