File: gauges/ClusterGauges.kicad_pcb (KiCad board)
At the start: 4 copper layers, 447.1 x 55.8 mm, 101 parts, among them J1 DTM06-3S nickel, 12V input + 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, J2 SWD Tag-Connect, J7 DTM06-5S nickel, CAN0 + 3x se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, J8 KK-254 22-27-2031, private li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, J9 KK-254 22-27-2021, Hall speed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, Q1 PMV55ENEA ideal diode (DGATE), Q2 PMV37ENEA automotive (AEC-Q10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, Q3 PMV55ENEA pass (HGATE), U1 NXP S32K144 automotive (AEC-Q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, U10 TCAN1044V-Q1 (AEC-Q100 G1), U2 LMR33630-Q1 (AEC-Q100 G1), U3 LM74930-Q1 (AEC-Q100 G1), U4 TLV733P-Q1 (AEC-Q100 G1), U5 NXP TJA1043T automotive CAN t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, U6 Raystar RFA401280B-AYW-DNF1 -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, U7 Raystar RFA401280B-AYW-DNF1 -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, U8 Raystar RFA401280B-AYW-DNF1 -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, U9 Raystar RFA401280B-AYW-DNF1 -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, Y1 8MHz (AEC-Q200)

Commit message: gauges rev C: six 12 V-active indicator-lamp inputs and a tach input
1966 Mustang lamps are 12 V-active (user-confirmed), tach input wanted.
- J10 (7-pin KK 254): left/right turn, high beam, brake, alternator, oil + GND.
  Each input: 33k/15k divider, BAV99-Q clamp, 10 nF filter, DNP 4.7k pull-up
  for a ground-switched lamp (firmware inverts that channel).
- J11 tach: two 18k 1206 (200 V) in series + 15k, 2.2 nF, clamp, DNP pull-up
  for open-collector outputs. Coil-negative use on a points system is not
  validated. MCU pins: tach = pin 57 (FTM1_CH5), lamps = pins 35/36/37/38/43/44.
- Protocol: Indicators (0x303), InputConfig (0x420), RpmFromTach status bit.
- Layout: new zone next to the MCU, battery divider moved next to the ADC.
  Sender ADC nets 242-348 mm -> 72-95 mm; lamp nets 75-97 mm, tach 103 mm.
- Catalog: 1206 200 V resistors and 2.2 nF (both PATTERN, confirm in cart).

ERC unchanged (4 known items), 0 unconnected, DRC accepted categories only.

Co-Authored-By: Claude Sonnet 5.5 <noreply@anthropic.com>
Parts:
- added C50: 10nF input filter, Left turn (AEC-Q200), Capacitor_SMD:C_0603_1608Metric, F.Cu at (299.7, 203.8)
- added C51: 10nF input filter, Right turn (AEC-Q200), Capacitor_SMD:C_0603_1608Metric, F.Cu at (293.6, 205.0)
- added C52: 10nF input filter, High beam (AEC-Q200), Capacitor_SMD:C_0603_1608Metric, F.Cu at (268.9, 206.6)
- added C53: 10nF input filter, Brake / parking brake (AEC-Q200), Capacitor_SMD:C_0603_1608Metric, F.Cu at (273.8, 207.0)
- added C54: 10nF input filter, Alternator / charge (AEC-Q200), Capacitor_SMD:C_0603_1608Metric, F.Cu at (278.8, 207.0)
- added C55: 10nF input filter, Oil pressure (AEC-Q200), Capacitor_SMD:C_0603_1608Metric, F.Cu at (258.9, 207.7)
- added C56: 2.2nF input filter, tach (AEC-Q200), Capacitor_SMD:C_0603_1608Metric, F.Cu at (263.9, 207.7)
- added D16: BAV99-Q input clamp, Left turn (AEC-Q101), Package_TO_SOT_SMD:SOT-23, F.Cu at (289.0, 187.5)
- added D17: BAV99-Q input clamp, Right turn (AEC-Q101), Package_TO_SOT_SMD:SOT-23, F.Cu at (294.8, 187.5)
- added D18: BAV99-Q input clamp, High beam (AEC-Q101), Package_TO_SOT_SMD:SOT-23, F.Cu at (289.0, 192.9)
- added D19: BAV99-Q input clamp, Brake / parking brake (AEC-Q101), Package_TO_SOT_SMD:SOT-23, F.Cu at (294.8, 192.9)
- added D20: BAV99-Q input clamp, Alternator / charge (AEC-Q101), Package_TO_SOT_SMD:SOT-23, F.Cu at (280.2, 195.6)
- added D21: BAV99-Q input clamp, Oil pressure (AEC-Q101), Package_TO_SOT_SMD:SOT-23, F.Cu at (259.4, 196.3)
- added D22: BAV99-Q input clamp, tach (AEC-Q101), Package_TO_SOT_SMD:SOT-23, F.Cu at (265.2, 196.3)
- added J10: KK-254 22-27-2071, indicator lamp inputs (6 x 12 V-active +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, Connector_Molex:Molex_KK-254_AE-6410-07A_1x07_P2.54mm_Vertical, F.Cu at (259.2, 189.3)
- added J11: KK-254 22-27-2021, tach input (signal + ground), Connector_Molex:Molex_KK-254_AE-6410-02A_1x02_P2.54mm_Vertical, F.Cu at (281.7, 190.2)
- added R58: 33k series, Left turn (AEC-Q200), Resistor_SMD:R_0603_1608Metric, F.Cu at (299.5, 193.9)
- added R59: 15k divider bottom, Left turn (AEC-Q200), Resistor_SMD:R_0603_1608Metric, F.Cu at (285.6, 197.4)
- added R60: 4.7k pull-up to VIN_PROT, DNP: fit only if the Left turn la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, Resistor_SMD:R_0603_1608Metric, F.Cu at (290.5, 197.4)
- added R61: 33k series, Right turn (AEC-Q200), Resistor_SMD:R_0603_1608Metric, F.Cu at (295.5, 198.1)
- added R62: 15k divider bottom, Right turn (AEC-Q200), Resistor_SMD:R_0603_1608Metric, F.Cu at (299.7, 198.8)
- added R63: 4.7k pull-up to VIN_PROT, DNP: fit only if the Right turn l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, Resistor_SMD:R_0603_1608Metric, F.Cu at (270.6, 199.6)
- added R64: 33k series, High beam (AEC-Q200), Resistor_SMD:R_0603_1608Metric, F.Cu at (275.6, 200.1)
- added R65: 15k divider bottom, High beam (AEC-Q200), Resistor_SMD:R_0603_1608Metric, F.Cu at (280.6, 200.1)
- added R66: 4.7k pull-up to VIN_PROT, DNP: fit only if the High beam la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, Resistor_SMD:R_0603_1608Metric, F.Cu at (258.9, 200.8)
- added R67: 33k series, Brake / parking brake (AEC-Q200), Resistor_SMD:R_0603_1608Metric, F.Cu at (263.9, 200.8)
- added R68: 15k divider bottom, Brake / parking brake (AEC-Q200), Resistor_SMD:R_0603_1608Metric, F.Cu at (285.5, 200.8)
- added R69: 4.7k pull-up to VIN_PROT, DNP: fit only if the Brake / park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, Resistor_SMD:R_0603_1608Metric, F.Cu at (290.5, 200.8)
- added R70: 33k series, Alternator / charge (AEC-Q200), Resistor_SMD:R_0603_1608Metric, F.Cu at (295.4, 201.6)
- added R71: 15k divider bottom, Alternator / charge (AEC-Q200), Resistor_SMD:R_0603_1608Metric, F.Cu at (268.9, 203.1)
- added R72: 4.7k pull-up to VIN_PROT, DNP: fit only if the Alternator /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, Resistor_SMD:R_0603_1608Metric, F.Cu at (273.8, 203.5)
- added R73: 33k series, Oil pressure (AEC-Q200), Resistor_SMD:R_0603_1608Metric, F.Cu at (278.8, 203.5)
- added R74: 15k divider bottom, Oil pressure (AEC-Q200), Resistor_SMD:R_0603_1608Metric, F.Cu at (258.9, 204.2)
- added R75: 4.7k pull-up to VIN_PROT, DNP: fit only if the Oil pressure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, Resistor_SMD:R_0603_1608Metric, F.Cu at (263.9, 204.2)
- added R76: 18k series, tach, 200V (AEC-Q200), Resistor_SMD:R_1206_3216Metric, F.Cu at (299.9, 188.1)
- added R77: 18k series, tach, 200V (AEC-Q200), Resistor_SMD:R_1206_3216Metric, F.Cu at (271.4, 195.8)
- added R78: 15k divider bottom, tach (AEC-Q200), Resistor_SMD:R_0603_1608Metric, F.Cu at (283.7, 204.3)
- added R79: 4.7k pull-up to VIN_PROT, DNP: fit only for an open-collect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, Resistor_SMD:R_0603_1608Metric, F.Cu at (288.7, 204.3)
- moved R42 173.7 mm to (164.2, 190.0)
- moved C6 159.6 mm to (357.4, 186.6)
- moved Y1 159.6 mm to (341.9, 187.6)
- moved C4 159.6 mm to (347.4, 186.6)
- moved J2 159.6 mm to (334.3, 187.8)
- moved U1 159.6 mm to (322.1, 192.5)
- moved C5 159.6 mm to (352.4, 186.6)
- moved R1 153.4 mm to (341.2, 192.1)
- moved C42 148.9 mm to (174.1, 186.6)
- moved C40 148.9 mm to (164.2, 186.6)
- moved J8 148.9 mm to (144.4, 189.3)
- moved R40 148.9 mm to (179.0, 186.6)
- moved U10 148.9 mm to (157.0, 188.6)
- moved C41 148.9 mm to (169.1, 186.6)
- moved R41 148.9 mm to (184.0, 186.6)
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Connections:
- U1 pad 35: (no net) -> LAMP_TURN_L
- U1 pad 36: (no net) -> LAMP_TURN_R
- U1 pad 37: (no net) -> LAMP_HIGH_BEAM
- U1 pad 38: (no net) -> LAMP_BRAKE
- U1 pad 43: (no net) -> LAMP_ALT
- U1 pad 44: (no net) -> LAMP_OIL
- U1 pad 57: (no net) -> TACH_IN
Routing:
- net ADC_BATT: track 356.5 -> 90.4 mm, vias 2 -> 3
- net ADC_TEMP: track 329.2 -> 72.5 mm, vias 2 -> 4
- net ADC_FUEL: track 342.7 -> 93.7 mm, vias 4 -> 3
- net ADC_OIL: track 343.7 -> 95.1 mm, vias 3 -> 4
- net AUX_DC0: track 74.9 -> 233.0 mm
- net AUX_DC2: track 246.7 -> 89.9 mm, vias 3 -> 2
- net AUX_CS3: track 348.4 -> 192.8 mm, vias 3 -> 2
- net AUX_DC3: track 344.1 -> 190.1 mm, vias 3 -> 4
- net AUX_CS2: track 252.2 -> 98.3 mm, vias 3 -> 2
- net AUX_CS0: track 82.5 -> 234.4 mm
- net GND: track 810.8 -> 941.5 mm, vias 23 -> 27
- net TACH_IN: track 0.00 -> 102.9 mm, vias 0 -> 5
- net LAMP_OIL: track 0.00 -> 96.5 mm, vias 0 -> 4
- net LAMP_ALT: track 0.00 -> 94.2 mm, vias 0 -> 5
- net BL_EN: track 262.1 -> 168.3 mm, vias 3 -> 2
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Other:
- board size 447.1 x 55.8 mm -> 447.1 x 58.3 mm

Commit message: gauges: dash dimmer input on J10 pin 8 (ADC0_SE7, pin 31)
The 1966 Mustang headlight switch dims the instrument lamps with a rheostat,
so the feed wire is 0 V with lights off and about 4-12 V when on. 22k/6.8k
divider, BAV99-Q clamp, 100 nF filter. J10 becomes 8-circuit (22-27-2081).
Protocol: Indicators gains DashLightsOn and DashDimmerPct. ERC unchanged (4),
0 unconnected, DRC accepted categories only, ADC nets 80-98 mm.

Co-Authored-By: Claude Sonnet 5.5 <noreply@anthropic.com>
Parts:
- added C57: 100nF input filter, dash dimmer (AEC-Q200), Capacitor_SMD:C_0603_1608Metric, F.Cu at (298.8, 210.1)
- added D23: BAV99-Q input clamp, dash dimmer (AEC-Q101), Package_TO_SOT_SMD:SOT-23, F.Cu at (288.7, 197.2)
- added R80: 22k divider top, dash dimmer (AEC-Q200), Resistor_SMD:R_0603_1608Metric, F.Cu at (298.8, 206.6)
- added R81: 6.8k divider bottom, dash dimmer (AEC-Q200), Resistor_SMD:R_0603_1608Metric, F.Cu at (278.9, 207.0)
- J10: value KK-254 22-27-2071, indicator lamp inputs (6 x 12 V-active + ground) -> KK-254 22-27-2081, indicator lamp inputs (6 x 12 V-active + ground) and dash-dimmer feed; footprint Connector_Molex:Molex_KK-254_AE-6410-07A_1x07_P2.54mm_Vertical -> Connector_Molex:Molex_KK-254_AE-6410-08A_1x08_P2.54mm_Vertical
- moved C50 40.8 mm to (259.1, 207.7), turned to 0 degrees
- moved D19 35.5 mm to (259.5, 196.3)
- moved C56 30.0 mm to (293.8, 210.1)
- moved C55 30.0 mm to (288.8, 210.1)
- moved C51 29.7 mm to (264.0, 207.7)
- moved R77 28.5 mm to (298.6, 187.0)
- moved R67 23.1 mm to (287.0, 201.6)
- moved R75 20.0 mm to (283.9, 205.1)
- moved R62 17.7 mm to (282.1, 200.1), turned to 0 degrees
- moved R70 16.6 mm to (278.9, 203.5)
- moved R66 15.0 mm to (274.0, 201.2)
- moved R74 15.0 mm to (274.0, 204.7)
- moved D20 14.8 mm to (265.4, 196.3)
- moved R59 13.5 mm to (299.1, 196.2)
- moved D21 11.9 mm to (271.2, 196.3)
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Connections:
- U1 pad 31: (no net) -> DIM_ADC
Routing:
- net DIM_ADC: track 0.00 -> 76.1 mm, vias 0 -> 4
- net TACH_MID: track 41.1 -> 3.64 mm, vias 2 -> 0
- net TACH_IN: track 102.9 -> 71.3 mm, vias 5 -> 4
- net LAMP_TURN_L: track 75.2 -> 106.2 mm
- net DIM_RAW: track 0.00 -> 28.4 mm, vias 0 -> 1
- net +3V3: track 632.2 -> 607.3 mm, vias 21 -> 18
- net LAMP_TURN_R: track 62.9 -> 86.0 mm, vias 4 -> 6
- net GND: track 941.5 -> 960.4 mm, vias 27 -> 24
- net IGN_SENSE: track 121.6 -> 109.2 mm
- net LAMP_HIGH_BEAM: track 69.0 -> 80.0 mm, vias 3 -> 4
- net CAN0_L: track 45.8 -> 35.9 mm
- net AUX_VLED_RTN: track 452.1 -> 442.7 mm, vias 5 -> 6
- net LAMP_OIL: track 96.5 -> 87.6 mm, vias 4 -> 5
- net VIN_FUSED: track 44.8 -> 53.6 mm
- net LAMP_BRAKE: track 87.7 -> 96.4 mm
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
Commit message: Add the physical turn-signal arrows to gauges/: two green LEDs lit straight from the flasher wires
ROHM CSL0902ET1C (AEC-Q102, land pattern from its data sheet) behind the faceplate, each from its LAMP_TURN_x_RAW wire through a 1.8k 1206 resistor, with a BAV99-Q reverse clamp, so they flash like the old bulbs and work with the software off. The J10 sense inputs are unchanged. X positions are placeholders from the concept drawing (TURN_LED_X in build_pcb.py) until the faceplate drawing exists. Re-routed to 0 unconnected nets (real kicad-cli DRC: same four accepted categories as before), BOM updated.

Co-Authored-By: Claude Sonnet 5.5 <noreply@anthropic.com>
Parts:
- added D24: BAV99-Q reverse clamp, Left turn arrow LED (AEC-Q101), Package_TO_SOT_SMD:SOT-23, F.Cu at (169.7, 229.8)
- added D25: BAV99-Q reverse clamp, Right turn arrow LED (AEC-Q101), Package_TO_SOT_SMD:SOT-23, F.Cu at (428.5, 229.8)
- added D26: CSL0902ET1C green LED, Left turn arrow, ROHM_CSL0902:CSL0902_1608, F.Cu at (165.3, 229.8)
- added D27: CSL0902ET1C green LED, Right turn arrow, ROHM_CSL0902:CSL0902_1608, F.Cu at (424.1, 229.8)
- added R82: 1.8k LED series, Left turn arrow (AEC-Q200), Resistor_SMD:R_1206_3216Metric, F.Cu at (159.7, 229.8)
- added R83: 1.8k LED series, Right turn arrow (AEC-Q200), Resistor_SMD:R_1206_3216Metric, F.Cu at (418.5, 229.8)
Routing:
- net LAMP_TURN_R_RAW: track 51.7 -> 195.0 mm, vias 2 -> 4
- net LAMP_TURN_L_RAW: track 43.0 -> 162.9 mm, vias 1 -> 2
- net GND: track 960.4 -> 1005.9 mm, vias 24 -> 22
- net VIN_PROT: track 472.6 -> 441.7 mm, vias 11 -> 15
- net LAMP_HIGH_BEAM: track 80.0 -> 104.2 mm, vias 4 -> 5
- net +3V3: track 607.3 -> 589.7 mm
- net AUX_DC0: track 232.5 -> 245.8 mm, vias 2 -> 3
- net AUX_CS0: track 238.9 -> 249.9 mm, vias 2 -> 3
- net AUX_RST: track 447.7 -> 458.6 mm, vias 7 -> 6
- net AUX_CS1: track 134.6 -> 144.7 mm
- net TURN_LED_L_A: track 0.00 -> 10.1 mm
- net TURN_LED_R_A: track 0.00 -> 10.1 mm
- net +5V: track 501.0 -> 509.9 mm
- net SENDER_OIL: track 59.4 -> 67.9 mm
- net CAN1_L: track 19.6 -> 27.6 mm, vias 1 -> 2
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
Commit message: Electrical design review: fix gauges J2 pinout and shorted crystal, MCU/CAN decoupling cells, connector TVS, extra input bulk; add review/ scripts and docs/electrical-review.md
Review scripts (review/): netlist vs datasheet pin tables, connector audit, ISO 7637 surge simulation, thermal/derating, DSI impedance, layout checks. gauges/ regenerated and routed: 0 unconnected nets, real DRC in the same four accepted categories. display/ reviewed read-only; its findings are open items in the report.

Co-Authored-By: Claude Sonnet 5.5 <noreply@anthropic.com>
Parts:
- added C58: 1uF X7R LDO input (AEC-Q200), Capacitor_SMD:C_0603_1608Metric, F.Cu at (126.5, 208.9)
- added C59: 10uF 50V X7S extra bulk at VIN_PROT (AEC-Q200), Capacitor_SMD:C_1210_3225Metric, F.Cu at (125.5, 188.1)
- added C60: 10uF 50V X7S extra bulk at VIN_PROT (AEC-Q200), Capacitor_SMD:C_1210_3225Metric, F.Cu at (122.8, 198.8)
- added D28: SM24CANB-02HTG TVS on the car CAN bus, at J7 (AEC-Q101), Package_TO_SOT_SMD:SOT-23, F.Cu at (422.7, 194.6)
- added D29: SM24CANB-02HTG TVS on the fuel and oil sender wires, at J7 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, Package_TO_SOT_SMD:SOT-23, F.Cu at (433.9, 187.8)
- added D30: SM24CANB-02HTG TVS on the coolant sender wire, at J7 (secon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, Package_TO_SOT_SMD:SOT-23, F.Cu at (443.3, 193.5)
- added D31: SM24CANB-02HTG TVS on the private CAN link, at J8 (AEC-Q101), Package_TO_SOT_SMD:SOT-23, F.Cu at (167.9, 191.3)
- added D32: SM24CANB-02HTG TVS on the Hall speed wire, at J9 (second ch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, Package_TO_SOT_SMD:SOT-23, F.Cu at (195.9, 190.1)
- added R84: 33R SPI SCK series termination at the MCU (AEC-Q200), Resistor_SMD:R_0603_1608Metric, F.Cu at (329.7, 206.9)
- added R85: 33R SPI MOSI series termination at the MCU (AEC-Q200), Resistor_SMD:R_0603_1608Metric, F.Cu at (327.7, 206.9)
- added R86: 100k BL_GATE pull-down, backlights stay off until firmware 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, Resistor_SMD:R_0603_1608Metric, F.Cu at (497.2, 186.6)
- added R87: 100k CAN0_EN pull-down, defined state while the MCU resets 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, Resistor_SMD:R_0603_1608Metric, F.Cu at (448.5, 199.2)
- added R88: 100k CAN0_STB_N pull-down, defined state while the MCU rese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, Resistor_SMD:R_0603_1608Metric, F.Cu at (457.7, 187.3)
- J2: value SWD Tag-Connect -> SWD Tag-Connect TC2030-IDC-NL (pin order per Tag-Connect: 1 VCC, 2 SWDIO, 3 nRESET, 4 SWCLK, 5 GND, 6 SWO)
- R16: value 1k fuel pull-up to +3V3 (11mW at a 10R sender) (AEC-Q200) -> 1k fuel pull-up to +3V3, 1206: a wire shorted to 14.4 V puts 123 mW in it (11mW at a 10R sender) (AEC-Q200); footprint Resistor_SMD:R_0603_1608Metric -> Resistor_SMD:R_1206_3216Metric
- R17: value 1k oil pull-up to +3V3 (AEC-Q200) -> 1k oil pull-up to +3V3, 1206 (AEC-Q200); footprint Resistor_SMD:R_0603_1608Metric -> Resistor_SMD:R_1206_3216Metric
- R18: value 1k coolant temp pull-up to +3V3 (AEC-Q200) -> 1k coolant temp pull-up to +3V3, 1206 (AEC-Q200); footprint Resistor_SMD:R_0603_1608Metric -> Resistor_SMD:R_1206_3216Metric
- moved R16 48.3 mm to (364.5, 187.0)
- moved C6 40.2 mm to (318.4, 197.1), turned to -90 degrees
- moved C5 39.2 mm to (316.4, 202.5), turned to -90 degrees
- moved L2 39.0 mm to (318.4, 193.7), turned to -90 degrees
- moved C4 36.6 mm to (312.6, 198.2), turned to -90 degrees
- moved C8 35.4 mm to (318.4, 200.5), turned to -90 degrees
- moved C31 34.5 mm to (373.6, 190.8)
- moved R19 34.5 mm to (363.7, 190.8)
- moved R20 34.5 mm to (368.7, 190.8)
- moved J8 30.6 mm to (174.9, 192.7), turned to 90 degrees
- moved C29 29.4 mm to (383.6, 192.0)
- moved C28 29.4 mm to (378.6, 192.0)
- moved Y1 28.4 mm to (315.5, 198.5), turned to -90 degrees
- moved R17 27.1 mm to (371.1, 187.0)
- moved R18 25.5 mm to (377.6, 187.0)
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Connections:
- J2 pad 1: SWDIO -> +3V3
- J2 pad 2: +3V3 -> SWDIO
- J2 pad 3: SWCLK -> RESET
- J2 pad 4: (no net) -> SWCLK
- J2 pad 5: RESET -> GND
- J2 pad 6: GND -> (no net)
- U1 pad 25: LPSPI2_SOUT -> LPSPI2_SOUT_MCU
- U1 pad 29: LPSPI2_SCK -> LPSPI2_SCK_MCU
- Y1 pad 2: OSC_OUT -> GND
- Y1 pad 3: OSC_IN -> OSC_OUT
- Y1 pad 4: OSC_OUT -> GND
Routing:
- net GND: track 1005.9 -> 1196.5 mm, vias 22 -> 26
- net +3V3: track 589.7 -> 643.6 mm, vias 18 -> 13
- net VIN_PROT: track 441.7 -> 474.5 mm, vias 15 -> 12
- net OSC_OUT: track 43.7 -> 11.5 mm, vias 3 -> 2
- net VDDA: track 45.1 -> 13.8 mm, vias 2 -> 3
- net ADC_BATT: track 88.5 -> 61.8 mm, vias 3 -> 4
- net IGN_RAW: track 136.3 -> 111.9 mm, vias 2 -> 1
- net OSC_IN: track 33.6 -> 9.86 mm, vias 2 -> 0
- net +5V: track 509.9 -> 487.3 mm, vias 10 -> 9
- net LAMP_TURN_R_RAW: track 195.0 -> 216.9 mm, vias 4 -> 3
- net CAN1_SPLIT: track 24.0 -> 3.82 mm
- net CAN0_SPLIT: track 30.6 -> 11.4 mm, vias 2 -> 0
- net TACH_IN: track 76.2 -> 95.4 mm, vias 4 -> 5
- net ADC_FUEL: track 91.9 -> 73.6 mm, vias 4 -> 3
- net CAN0_H: track 28.9 -> 46.9 mm
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