File: gauges/ClusterGauges.kicad_pcb (KiCad board)
At the start: 4 copper layers, 447.1 x 58.3 mm, 162 parts, among them J1 DTM06-3S nickel, 12V input + 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, J10 KK-254 22-27-2081, indicator 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, J11 KK-254 22-27-2021, tach input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, J2 SWD Tag-Connect TC2030-IDC-NL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, J7 DTM06-5S nickel, CAN0 + 3x se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, J8 KK-254 22-27-2031, private li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, J9 KK-254 22-27-2021, Hall speed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, Q1 PMV55ENEA ideal diode (DGATE), Q2 PMV37ENEA automotive (AEC-Q10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, Q3 PMV55ENEA pass (HGATE), U1 NXP S32K144 automotive (AEC-Q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, U10 TCAN1044V-Q1 (AEC-Q100 G1), U2 LMR33630-Q1 (AEC-Q100 G1), U3 LM74930-Q1 (AEC-Q100 G1), U4 TLV733P-Q1 (AEC-Q100 G1), U5 NXP TJA1043T automotive CAN t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, U6 Raystar RFA401280B-AYW-DNF1 -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, U7 Raystar RFA401280B-AYW-DNF1 -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, U8 Raystar RFA401280B-AYW-DNF1 -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, U9 Raystar RFA401280B-AYW-DNF1 -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, Y1 8MHz (AEC-Q200)

Commit message: Electrical review, part 2: +3V3 rail clamp on gauges, display battery path and TVS footprint, harness wording, new display parts reviewed
gauges/: D33 (onsemi SZMMSZ3V6T1G 3.6 V zener) clamps +3V3 when a sender wire is shorted to battery with the car off (G-08); BOM and connector values follow docs/harness.md (J7 DTM06-6S with a sealed cavity, J8 an in-dash KK 254 cable, 20/22 AWG). display/: D1 footprint D_SMB -> D_SMC to match the SMCJ33A in the BOM (D-01); VBAT_IN, VBAT_F, SENSE_OUT and COMMON added to TRUNK_NETS (D-02). review/expected.py covers the TAC5112-Q1, TPS2557-Q1, TPD4E05U06-Q1 and the second TLV767-Q1. Both boards regenerated and routed: real kicad-cli DRC 0 unconnected, only accepted categories; fab packages rebuilt.

Co-Authored-By: Claude Opus 5.5 <noreply@anthropic.com>
Parts:
- added D33: SZMMSZ3V6T1G 3.6V zener clamp on +3V3, absorbs a sender wir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, Diode_SMD:D_SOD-123, F.Cu at (387.7, 187.0)
- J1: value DTM06-3S nickel, 12V input + ignition (sealed) -> Phoenix MKDS 1,5/3-5,08: 12V, GND, ignition (20 AWG GXL pigtail, DTM06-3S plug on the car end)
- J10: value KK-254 22-27-2081, indicator lamp inputs (6 x 12 V-active + ground) and dash-dimmer feed -> KK-254 22-27-2081, indicator lamp inputs (6 x 12 V-active + ground) and dash-dimmer feed (22 AWG pigtail, DTM06-08SA pl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
- J11: value KK-254 22-27-2021, tach input (signal + ground) -> KK-254 22-27-2021, tach input (signal + ground; 22 AWG pigtail, DTM06-2S plug)
- J7: value DTM06-5S nickel, CAN0 + 3x sender input (sealed) -> KK-254 22-27-2051: CAN0 + 3 sender inputs (22 AWG pigtail, DTM06-6S plug with one cavity sealed)
- J8: value KK-254 22-27-2031, private link to display/ J3 (DTM06-3S pigtail) -> KK-254 22-27-2031, private CAN link to display/ J3 (in-dash KK 254 cable, 22 AWG twisted pair + ground, no DTM)
- J9: value KK-254 22-27-2021, Hall speed sender (signal + ground) -> KK-254 22-27-2021, Hall speed sender (signal + ground; 22 AWG pigtail, DTM06-2S plug)
- moved R19 36.4 mm to (400.1, 190.8)
- moved R16 29.8 mm to (394.3, 187.0)
- moved R17 29.8 mm to (400.9, 187.0)
- moved D15 20.0 mm to (363.8, 187.5)
- moved D12 20.0 mm to (369.7, 187.5)
- moved D13 20.0 mm to (375.6, 187.5)
- moved D14 20.0 mm to (381.4, 187.5)
- moved R20 18.2 mm to (386.8, 190.9)
- moved R18 17.2 mm to (394.3, 191.2)
- moved R56 16.0 mm to (382.5, 192.7), turned to 90 degrees
- moved R55 10.8 mm to (404.3, 191.6), turned to 90 degrees
- moved C31 10.3 mm to (363.4, 192.0)
- moved C28 10.2 mm to (368.4, 192.0)
- moved C29 10.2 mm to (373.3, 192.0)
- moved C30 10.2 mm to (378.3, 192.0)
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Routing:
- net ADC_FUEL: track 73.6 -> 121.8 mm, vias 3 -> 4
- net GND: track 1196.5 -> 1164.6 mm, vias 26 -> 29
- net SENDER_FUEL: track 77.7 -> 49.8 mm, vias 3 -> 2
- net ADC_OIL: track 81.0 -> 58.7 mm, vias 3 -> 4
- net VIN_PROT: track 474.5 -> 452.7 mm, vias 12 -> 11
- net AUX_DC1: track 140.9 -> 162.7 mm
- net SENDER_TEMP: track 72.7 -> 53.2 mm, vias 2 -> 1
- net LAMP_TURN_R_RAW: track 216.9 -> 200.0 mm
- net ADC_BATT: track 61.8 -> 77.4 mm, vias 4 -> 0
- net AUX_DC0: track 241.3 -> 256.3 mm, vias 3 -> 2
- net LPSPI2_SCK: track 434.1 -> 419.3 mm
- net LAMP_OIL: track 91.6 -> 106.3 mm
- net AUX_VLED_RTN: track 444.0 -> 458.5 mm
- net AUX_CS0: track 240.2 -> 254.6 mm, vias 4 -> 2
- net LAMP_BRAKE: track 111.8 -> 97.8 mm
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
Commit message: Fix what would stop the boards becoming a product: Verdin mounting, FETs, CarPlay header
Product review 2026-10-18 (docs/electrical-review.md section 8a):
- display: Toradex's four M2 standoffs (S1/S2 2.5 mm module hold-down for
  vibration, S3/S4 7.0 mm for the Verdin Industrial Heatsink) at the design
  guide's Fig 113 positions, GND rings kept on the outer layers; the module
  keepout now follows the real module outline (the module is not centred
  on the socket; the strip under its far edge was open). 178.2 x 105.0 mm.
- display: J16 is a 1x6 MFi daughterboard header with a 5 V supply switched
  by U15 (TPS22918-Q1) from Verdin GPIO_3, as LIVI's carPlayMfiPowerGpio
  expects; the Apple part itself stays on the daughterboard (NDA).
- both: the LM74930 FET pair is Vishay SQJ460AEP (PowerPAK SO-8L, 8.7 mohm,
  IDM 180 A) instead of the NRND SOT-23 PMV55ENEA (X-01, X-02, D-05).
- gauges: 2.2 uH XAL5030-222MEC and 16 V 1210 output caps per the LMR33630
  datasheet (G-14), 1 uF CVS (G-17); inner small gauges at the measured
  +/-118 mm (owner photos), arrows midway between each side's gauges.
- display: 16 V 1210 panel-bias output caps (D-03); bidirectional
  TPD4E02B04-Q1 on the line-out legs (D-11).
- docs: depth stack-up first pass, Toradex supply/thermal/BSP questions,
  an RFQ for wider-temperature small displays, BOM supply-risk note.
Both boards: 0 unconnected, DRC only in the accepted categories, BOM
coverage and fab gate pass; review_netlist gauges 62/62, display only the
pre-existing U6 decoupling distance.

Co-Authored-By: Claude Opus 5.5 <noreply@anthropic.com>
Parts:
- C2, C45: value 22uF 10V X7R COUT (AEC-Q200) -> 22uF 16V X7R COUT (AEC-Q200); footprint Capacitor_SMD:C_1206_3216Metric -> Capacitor_SMD:C_1210_3225Metric
- C47: value 100nF CVS (50V) -> 1uF CVS (50V); footprint Capacitor_SMD:C_0603_1608Metric -> Capacitor_SMD:C_0805_2012Metric
- L1: value 10uH power XAL5050-103ME (AEC-Q200) -> 2.2uH power XAL5030-222ME (AEC-Q200); footprint Inductor_SMD:L_Coilcraft_XAL5050-XXX -> Inductor_SMD:L_Coilcraft_XAL5030-XXX
- Q1: value PMV55ENEA ideal diode (DGATE) -> SQJ460AEP ideal diode (DGATE); footprint Package_TO_SOT_SMD:SOT-23 -> Package_SO:PowerPAK_SO-8L_Single
- Q3: value PMV55ENEA pass (HGATE) -> SQJ460AEP pass (HGATE); footprint Package_TO_SOT_SMD:SOT-23 -> Package_SO:PowerPAK_SO-8L_Single
- moved D24 28.7 mm to (141.1, 232.3)
- moved D26 28.7 mm to (136.7, 232.3)
- moved R82 28.7 mm to (131.1, 232.3)
- moved D25 27.6 mm to (455.9, 232.3)
- moved D27 27.6 mm to (451.6, 232.3)
- moved R83 27.6 mm to (445.9, 232.3)
- moved U7 19.7 mm to (176.0, 232.9)
- moved C18 19.7 mm to (178.5, 224.3)
- moved R7 19.7 mm to (173.5, 224.3)
- moved U8 19.7 mm to (412.0, 232.9)
- moved C19 19.7 mm to (414.5, 224.3)
- moved R8 19.7 mm to (409.5, 224.3)
- moved C2 18.3 mm to (130.4, 201.5), turned to 0 degrees
- moved Q3 17.4 mm to (112.0, 194.4), turned to 0 degrees
- moved R48 16.6 mm to (107.3, 188.9), turned to -90 degrees
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Connections:
- Q1 pad 1: DGATE -> COMMON
- Q1 pad 3: VIN_PROT -> COMMON
- Q3 pad 1: HGATE -> COMMON
- Q3 pad 3: SENSE_OUT -> COMMON
Routing:
- net GND: track 1164.6 -> 1203.4 mm, vias 29 -> 27
- net ADC_FUEL: track 121.8 -> 84.3 mm
- net LAMP_BRAKE: track 97.8 -> 130.2 mm
- net LAMP_TURN_L_RAW: track 163.1 -> 193.2 mm, vias 2 -> 4
- net AUX_CS2: track 84.0 -> 113.1 mm
- net LAMP_TURN_R: track 95.6 -> 122.6 mm, vias 6 -> 4
- net AUX_DC2: track 80.9 -> 103.6 mm, vias 3 -> 2
- net LAMP_TURN_L: track 105.4 -> 125.9 mm, vias 5 -> 3
- net TACH_IN: track 102.3 -> 85.4 mm
- net LAMP_TURN_R_RAW: track 200.0 -> 216.8 mm, vias 3 -> 4
- net AUX_CS1: track 144.4 -> 160.0 mm, vias 4 -> 2
- net SENSE_OUT: track 9.70 -> 25.1 mm, vias 0 -> 2
- net DIM_ADC: track 95.3 -> 80.8 mm, vias 4 -> 5
- net LAMP_ALT: track 112.8 -> 126.8 mm
- net AUX_DC0: track 256.3 -> 242.4 mm, vias 2 -> 3
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Other:
- board size 447.1 x 58.3 mm -> 447.1 x 63.4 mm

Commit message: Six layers with solid GND planes, a field-solved DSI geometry, and the RGB variant routed
Both boards and display-rgb/ move to JLC06161H-3313 six-layer: F / In1 GND /
In2 / In3 with the +5V or +3V3 pour / In4 GND / B. Every net class except GND
is restricted to F, In2, In3 and B in the router input (FreeRouting 2.2.4
ignores a layer_rule "active off"), and review/layout_checks.py now fails a
board with any track on In1 or In4. All three boards: 0 unconnected under
kicad-cli DRC, accepted categories only, no copper but GND fill on the planes.

- DSI pairs are 0.16 mm, field-solved on the new stack-up at 96.4-103.1 ohm
  differential (review/dsi_impedance.py); board minimum track 0.15 mm.
- gauges/ routes VIN_PROT, VIN_FUSED and +5V at 0.4 mm from the start; every
  power net now passes the 20 K current check, and nothing crosses the buck's
  switch node (P-07).
- Panel bias +5.98 V / -6.05 V, inside the ICNL9707's rating; fab/README.md
  gives a diode-test check of the panel's pin polarity before JP1/JP2.
- display-rgb/ brought up to date with display/ (standoffs, FETs, audio,
  USB-C, MFi header), RGB parts renumbered, routed; still not a fab candidate
  while its panel connector is a placeholder.
- FreeRouting runs end at routing: (postroute off) in the DSN, a job timeout
  as backstop; one in-place attempt, since retries of one DSN are identical.
- The OV/UV divider tops are pulled to the LM74930 SW pin.
- docs/electrical-review.md section 8b records the measured results; the
  display/ battery path on inner copper (D-02 residual) is still open.

Co-Authored-By: Claude Opus 5.5 <noreply@anthropic.com>
Parts:
- moved D1 17.6 mm to (105.7, 200.1), turned to 0 degrees
- moved R54 10.9 mm to (92.3, 196.1), turned to 180 degrees
- moved R53 8.86 mm to (93.8, 194.2)
- moved C48 4.61 mm to (98.4, 184.8)
- moved Q3 4.61 mm to (109.9, 190.3)
- moved R48 4.61 mm to (105.2, 184.8)
- moved C47 4.61 mm to (99.3, 196.6)
- moved R49 4.61 mm to (101.8, 185.2)
- moved R50 4.61 mm to (105.6, 195.6)
- moved R51 4.61 mm to (96.4, 195.0), turned to -90 degrees
- moved C49 4.61 mm to (102.2, 195.6)
- moved Q1 4.61 mm to (93.2, 189.7)
- moved U3 4.61 mm to (101.7, 190.6)
- moved C11 2.17 mm to (128.2, 195.0)
- moved C12 2.17 mm to (126.7, 186.2)
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Routing:
- net GND: track 1203.4 -> 196.9 mm, vias 27 -> 111
- net LAMP_BRAKE: track 130.2 -> 99.4 mm
- net LAMP_TURN_R_RAW: track 216.8 -> 242.2 mm
- net LAMP_TURN_R: track 122.6 -> 101.3 mm, vias 4 -> 6
- net AUX_CS3: track 184.9 -> 206.1 mm
- net DIM_ADC: track 80.8 -> 99.7 mm, vias 5 -> 4
- net LAMP_TURN_L: track 125.9 -> 107.1 mm, vias 3 -> 4
- net LAMP_ALT: track 126.8 -> 110.2 mm, vias 6 -> 5
- net LPSPI2_SOUT: track 428.5 -> 442.8 mm, vias 7 -> 6
- net AUX_RST: track 459.0 -> 447.8 mm
- net LAMP_HIGH_BEAM: track 89.0 -> 99.4 mm
- net LAMP_BRAKE_RAW: track 39.6 -> 49.3 mm
- net SW: track 9.37 -> 16.1 mm, vias 0 -> 2
- net VIN_FUSED: track 51.7 -> 58.2 mm, vias 2 -> 4
- net U6_VLED: track 11.9 -> 5.95 mm
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- added copper zone on In3.Cu, net +3V3
- added copper zone on In2.Cu, net GND
- added copper zone on In4.Cu, net GND
- removed copper zone on In2.Cu, net +3V3
Other:
- copper layers 4 -> 6
