File: gauges/ClusterGauges.kicad_sch (KiCad schematic)
At the start: 156 parts, among them J1 DTM06-3S nickel, 12V input + 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, J10 KK-254 22-27-2081, indicator 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, J11 KK-254 22-27-2021, tach input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, J2 SWD Tag-Connect TC2030-IDC-NL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, J7 DTM06-5S nickel, CAN0 + 3x se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, J8 KK-254 22-27-2031, private li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, J9 KK-254 22-27-2021, Hall speed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, Q1 PMV55ENEA ideal diode (DGATE), Q2 PMV37ENEA automotive (AEC-Q10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, Q3 PMV55ENEA pass (HGATE), U1 NXP S32K144 automotive (AEC-Q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, U10 TCAN1044V-Q1 (AEC-Q100 G1), U2 LMR33630-Q1 (AEC-Q100 G1), U3 LM74930-Q1 (AEC-Q100 G1), U4 TLV733P-Q1 (AEC-Q100 G1), U5 NXP TJA1043T automotive CAN t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, U6 Raystar RFA401280B-AYW-DNF1 -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, U7 Raystar RFA401280B-AYW-DNF1 -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, U8 Raystar RFA401280B-AYW-DNF1 -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, U9 Raystar RFA401280B-AYW-DNF1 -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, Y1 8MHz (AEC-Q200)

Commit message: Electrical review, part 2: +3V3 rail clamp on gauges, display battery path and TVS footprint, harness wording, new display parts reviewed
gauges/: D33 (onsemi SZMMSZ3V6T1G 3.6 V zener) clamps +3V3 when a sender wire is shorted to battery with the car off (G-08); BOM and connector values follow docs/harness.md (J7 DTM06-6S with a sealed cavity, J8 an in-dash KK 254 cable, 20/22 AWG). display/: D1 footprint D_SMB -> D_SMC to match the SMCJ33A in the BOM (D-01); VBAT_IN, VBAT_F, SENSE_OUT and COMMON added to TRUNK_NETS (D-02). review/expected.py covers the TAC5112-Q1, TPS2557-Q1, TPD4E05U06-Q1 and the second TLV767-Q1. Both boards regenerated and routed: real kicad-cli DRC 0 unconnected, only accepted categories; fab packages rebuilt.

Co-Authored-By: Claude Opus 5.5 <noreply@anthropic.com>
Parts:
- added D33: SZMMSZ3V6T1G 3.6V zener clamp on +3V3, absorbs a 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, Diode_SMD:D_SOD-123, symbol ClusterGauges:ZENER
- J1: value DTM06-3S nickel, 12V input + ignition (sealed) -> Phoenix MKDS 1,5/3-5,08: 12V, GND, ignition (20 AWG GXL pigtail, DTM06-3S plug on the car end)
- J10: value KK-254 22-27-2081, indicator lamp inputs (6 x 12 V-active + ground) and dash-dimmer feed -> KK-254 22-27-2081, indicator lamp inputs (6 x 12 V-active + ground) and dash-dimmer feed (22 AWG pigtail, DTM06-08SA pl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
- J11: value KK-254 22-27-2021, tach input (signal + ground) -> KK-254 22-27-2021, tach input (signal + ground; 22 AWG pigtail, DTM06-2S plug)
- J7: value DTM06-5S nickel, CAN0 + 3x sender input (sealed) -> KK-254 22-27-2051: CAN0 + 3 sender inputs (22 AWG pigtail, DTM06-6S plug with one cavity sealed)
- J8: value KK-254 22-27-2031, private link to display/ J3 (DTM06-3S pigtail) -> KK-254 22-27-2031, private CAN link to display/ J3 (in-dash KK 254 cable, 22 AWG twisted pair + ground, no DTM)
- J9: value KK-254 22-27-2021, Hall speed sender (signal + ground) -> KK-254 22-27-2021, Hall speed sender (signal + ground; 22 AWG pigtail, DTM06-2S plug)
Connections:
- net +3V3: now also D33.1 (K)
- net GND: now also D33.2 (A)
Other:
- note added: "6. Harness (decided 2026-10-17, docs/harness.md): J1 Phoenix MKDS with a 20 AWG GXL"
- note added: "DTM06-6S / -2S / -08SA / -2S plugs; J8 an in-dash KK 254 cable to display/ J3."
- note added: "No sealed connector is mounted on the board."
- note added: "pigtail and DTM06-3S plug; J7/J9/J10/J11 KK 254 headers with 22 AWG pigtails and"
- note removed: "6. J1 (power) and J7 (CAN0 + 3x sender) both land real Molex KK-254/Phoenix MKDS"
- note removed: "board-side connectors, sealed DTM06 nickel pigtails on the outboard end - same"
- note removed: "for a dash-mounted (not engine-bay) board."
- note removed: "real strategy thermo-pcb established. Not yet re-confirmed as the right choice"
