File: gauges/ClusterGauges.kicad_sch (KiCad schematic)
At the start: 157 parts, among them J1 Phoenix MKDS 1,5/3-5,08: 12V,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, J10 KK-254 22-27-2081, indicator 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, J11 KK-254 22-27-2021, tach input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, J2 SWD Tag-Connect TC2030-IDC-NL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, J7 KK-254 22-27-2051: CAN0 + 3 s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, J8 KK-254 22-27-2031, private CA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, J9 KK-254 22-27-2021, Hall speed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, Q1 PMV55ENEA ideal diode (DGATE), Q2 PMV37ENEA automotive (AEC-Q10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, Q3 PMV55ENEA pass (HGATE), U1 NXP S32K144 automotive (AEC-Q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, U10 TCAN1044V-Q1 (AEC-Q100 G1), U2 LMR33630-Q1 (AEC-Q100 G1), U3 LM74930-Q1 (AEC-Q100 G1), U4 TLV733P-Q1 (AEC-Q100 G1), U5 NXP TJA1043T automotive CAN t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, U6 Raystar RFA401280B-AYW-DNF1 -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, U7 Raystar RFA401280B-AYW-DNF1 -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, U8 Raystar RFA401280B-AYW-DNF1 -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, U9 Raystar RFA401280B-AYW-DNF1 -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, Y1 8MHz (AEC-Q200)

Commit message: Fix what would stop the boards becoming a product: Verdin mounting, FETs, CarPlay header
Product review 2026-10-18 (docs/electrical-review.md section 8a):
- display: Toradex's four M2 standoffs (S1/S2 2.5 mm module hold-down for
  vibration, S3/S4 7.0 mm for the Verdin Industrial Heatsink) at the design
  guide's Fig 113 positions, GND rings kept on the outer layers; the module
  keepout now follows the real module outline (the module is not centred
  on the socket; the strip under its far edge was open). 178.2 x 105.0 mm.
- display: J16 is a 1x6 MFi daughterboard header with a 5 V supply switched
  by U15 (TPS22918-Q1) from Verdin GPIO_3, as LIVI's carPlayMfiPowerGpio
  expects; the Apple part itself stays on the daughterboard (NDA).
- both: the LM74930 FET pair is Vishay SQJ460AEP (PowerPAK SO-8L, 8.7 mohm,
  IDM 180 A) instead of the NRND SOT-23 PMV55ENEA (X-01, X-02, D-05).
- gauges: 2.2 uH XAL5030-222MEC and 16 V 1210 output caps per the LMR33630
  datasheet (G-14), 1 uF CVS (G-17); inner small gauges at the measured
  +/-118 mm (owner photos), arrows midway between each side's gauges.
- display: 16 V 1210 panel-bias output caps (D-03); bidirectional
  TPD4E02B04-Q1 on the line-out legs (D-11).
- docs: depth stack-up first pass, Toradex supply/thermal/BSP questions,
  an RFQ for wider-temperature small displays, BOM supply-risk note.
Both boards: 0 unconnected, DRC only in the accepted categories, BOM
coverage and fab gate pass; review_netlist gauges 62/62, display only the
pre-existing U6 decoupling distance.

Co-Authored-By: Claude Opus 5.5 <noreply@anthropic.com>
Parts:
- removed C2, C45: 22uF 10V X7R COUT (AEC-Q200), Capacitor_SMD:C_1206_3216Metric, symbol ClusterGauges:C_1206
- removed C47: 100nF CVS (50V), Capacitor_SMD:C_0603_1608Metric, symbol ClusterGauges:C_V
- removed Q1: PMV55ENEA ideal diode (DGATE), Package_TO_SOT_SMD:SOT-23, symbol ClusterGauges:MOSFET_N55
- removed Q3: PMV55ENEA pass (HGATE), Package_TO_SOT_SMD:SOT-23, symbol ClusterGauges:MOSFET_N55
- added C2, C45: 22uF 16V X7R COUT (AEC-Q200), Capacitor_SMD:C_1210_3225Metric, symbol ClusterGauges:C_1210
- added C47: 1uF CVS (50V), Capacitor_SMD:C_0805_2012Metric, symbol ClusterGauges:C_0805
- added Q1: SQJ460AEP ideal diode (DGATE), Package_SO:PowerPAK_SO-8L_Single, symbol ClusterGauges:MOSFET_PWR
- added Q3: SQJ460AEP pass (HGATE), Package_SO:PowerPAK_SO-8L_Single, symbol ClusterGauges:MOSFET_PWR
- L1: value 10uH power XAL5050-103ME (AEC-Q200) -> 2.2uH power XAL5030-222ME (AEC-Q200); footprint Inductor_SMD:L_Coilcraft_XAL5050-XXX -> Inductor_SMD:L_Coilcraft_XAL5030-XXX
Connections:
- net +5V: now also C2.1, C45.1
- net COMMON: now also Q1.1 (S), Q1.2 (S), Q1.3 (S), Q3.1 (S), Q3.2 (S), Q3.3 (S)
- net DGATE: now also Q1.4 (G)
- net GND: now also C2.2, C45.2, C47.2
- net HGATE: now also Q3.4 (G)
- net SENSE_OUT: now also Q3.5 (D)
- net VIN_FUSED: now also C47.1
- net VIN_PROT: now also Q1.5 (D)
