File: display/ClusterDisplay.kicad_sch (KiCad schematic)
At the start: 160 parts, among them J1 Verdin iMX95 Hexa 8GB WB IT, J10 RTC coin cell, J11 Molex KK-254 22-27-2041, rota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, J12 Samtec TSW-103-07-G-S A55 con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, J13 Samtec TSW-105-07-G-S USB_1 O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, J14 JST XH B5B-XH-A balanced line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, J15 JST XH B3B-XH-A electret micr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, J16 MFi coprocessor access I2C_1 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, J17 GCT USB4105-GF-A USB-C 2.0 ho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, J2 Phoenix MKDS 1,5/3-5,08 power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, J3 Molex KK-254 22-27-2031 priva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, J4 TST040HDBC-42 panel, J8 Samtec TSW-108-07-G-S JTAG (b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, J9 Samtec TSW-104-07-G-S buttons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, Q1 PMV55ENEA (AEC-Q101, 60V/20V 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, Q2 PMV55ENEA (AEC-Q101, 60V/20V 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, Q3 PMV55ENEA ignition wake pulld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, U1 LM74930-Q1, U10 TLV767-Q1 (3.3 V audio AVDD), U11 TPS2557-Q1, U12 TPD4E05U06-Q1 line-out ESD, U13 TPD4E05U06-Q1 mic ESD, U14 TPD4E05U06-Q1 USB ESD, U2 LM61460-Q1, U3 TLV767-Q1, U4 TCAN1044V-Q1, U6 TPS65131-Q1, U7 TPS61165-Q1, U8 TPS22918-Q1 (AEC-Q100 G2) dia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, U9 TAC5112-Q1

Commit message: Fix what would stop the boards becoming a product: Verdin mounting, FETs, CarPlay header
Product review 2026-10-18 (docs/electrical-review.md section 8a):
- display: Toradex's four M2 standoffs (S1/S2 2.5 mm module hold-down for
  vibration, S3/S4 7.0 mm for the Verdin Industrial Heatsink) at the design
  guide's Fig 113 positions, GND rings kept on the outer layers; the module
  keepout now follows the real module outline (the module is not centred
  on the socket; the strip under its far edge was open). 178.2 x 105.0 mm.
- display: J16 is a 1x6 MFi daughterboard header with a 5 V supply switched
  by U15 (TPS22918-Q1) from Verdin GPIO_3, as LIVI's carPlayMfiPowerGpio
  expects; the Apple part itself stays on the daughterboard (NDA).
- both: the LM74930 FET pair is Vishay SQJ460AEP (PowerPAK SO-8L, 8.7 mohm,
  IDM 180 A) instead of the NRND SOT-23 PMV55ENEA (X-01, X-02, D-05).
- gauges: 2.2 uH XAL5030-222MEC and 16 V 1210 output caps per the LMR33630
  datasheet (G-14), 1 uF CVS (G-17); inner small gauges at the measured
  +/-118 mm (owner photos), arrows midway between each side's gauges.
- display: 16 V 1210 panel-bias output caps (D-03); bidirectional
  TPD4E02B04-Q1 on the line-out legs (D-11).
- docs: depth stack-up first pass, Toradex supply/thermal/BSP questions,
  an RFQ for wider-temperature small displays, BOM supply-risk note.
Both boards: 0 unconnected, DRC only in the accepted categories, BOM
coverage and fab gate pass; review_netlist gauges 62/62, display only the
pre-existing U6 decoupling distance.

Co-Authored-By: Claude Opus 5.5 <noreply@anthropic.com>
Parts:
- removed C46: 22u VPOS out 16V (AEC-Q200), Capacitor_SMD:C_1206_3216Metric, symbol ClusterDisplay:C_1206
- removed C47: 22u VNEG out 16V (AEC-Q200), Capacitor_SMD:C_1206_3216Metric, symbol ClusterDisplay:C_1206
- removed Q1: PMV55ENEA (AEC-Q101, 60V/20V VGS) diode, Package_TO_SOT_SMD:SOT-23, symbol ClusterDisplay:NFET
- removed Q2: PMV55ENEA (AEC-Q101, 60V/20V VGS) pass, Package_TO_SOT_SMD:SOT-23, symbol ClusterDisplay:NFET
- removed U12: TPD4E05U06-Q1 line-out ESD, Package_SON:USON-10_2.5x1.0mm_P0.5mm, symbol ClusterDisplay:TPD4E05U06-Q1
- added C46: 22u VPOS out 16V (AEC-Q200), Capacitor_SMD:C_1210_3225Metric, symbol ClusterDisplay:C_1210
- added C47: 22u VNEG out 16V (AEC-Q200), Capacitor_SMD:C_1210_3225Metric, symbol ClusterDisplay:C_1210
- added C83: 1u MFi switch CIN, Capacitor_SMD:C_0603_1608Metric, symbol ClusterDisplay:C
- added C84: 1u MFi 5V out, Capacitor_SMD:C_0603_1608Metric, symbol ClusterDisplay:C
- added Q1: SQJ460AEP (AEC-Q101, 60V/20V VGS) diode, Package_SO:PowerPAK_SO-8L_Single, symbol ClusterDisplay:NFET_PWR
- added Q2: SQJ460AEP (AEC-Q101, 60V/20V VGS) pass, Package_SO:PowerPAK_SO-8L_Single, symbol ClusterDisplay:NFET_PWR
- added R74: 100k MFi switch off in reset, Resistor_SMD:R_0603_1608Metric, symbol ClusterDisplay:R
- added U12: TPD4E02B04-Q1 line-out ESD (bidirectional, review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, Package_SON:USON-10_2.5x1.0mm_P0.5mm, symbol ClusterDisplay:TPD4E02B04-Q1
- added U15: TPS22918-Q1 (AEC-Q100 G2) MFi 5V switch, Package_TO_SOT_SMD:SOT-23-6, symbol ClusterDisplay:TPS22918-Q1
- J16: value MFi coprocessor access I2C_1 + reset (TBD, DNP) -> MFi daughterboard header I2C_1, reset, switched 5V, 1V8 (DNP); footprint Connector_PinHeader_2.54mm:PinHeader_1x04_P2.54mm_Vertical -> Connector_PinHeader_2.54mm:PinHeader_1x06_P2.54mm_Vertical
Connections:
- net +12V_PROT: now also Q1.5 (D)
- net +1V8: now also J16.6 (V1V8)
- net +5V: now also C83.1, U15.1 (VIN)
- net COMMON: now also Q1.1 (S1), Q1.2 (S2), Q1.3 (S3), Q2.1 (S1), Q2.2 (S2), Q2.3 (S3)
- net DGATE: now also Q1.4 (G)
- net GND: now also C46.2, C47.2, C83.2, C84.2, R74.2, U12.3 (GND1), U12.8 (GND2), U15.2 (GND)
- net HGATE: now also Q2.4 (G)
- net LINE_L_N: now also U12.2 (CH2)
- net LINE_L_P: now also U12.1 (CH1)
- net LINE_R_N: now also U12.5 (CH4)
- net LINE_R_P: now also U12.4 (CH3)
- net PANEL_VSN: now also C47.1
- net PANEL_VSP: now also C46.1
- net SENSE_OUT: now also Q2.5 (D)
- net MFI_PWR_EN: now reaches J1.210 (GPIO_3)
- net MFI_PWR_EN: now also R74.1, U15.3 (ON)
- new net MFI_5V: C84.1, J16.5 (VSW), U15.6 (VOUT)
- no-connect marks 205 -> 206
