File: display/ClusterDisplay.kicad_sch (KiCad schematic)
At the start: 164 parts, among them J1 Verdin iMX95 Hexa 8GB WB IT, J10 RTC coin cell, J11 Molex KK-254 22-27-2041, rota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, J12 Samtec TSW-103-07-G-S A55 con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, J13 Samtec TSW-105-07-G-S USB_1 O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, J14 JST XH B5B-XH-A balanced line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, J15 JST XH B3B-XH-A electret micr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, J16 MFi daughterboard header I2C_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, J17 GCT USB4105-GF-A USB-C 2.0 ho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, J2 Phoenix MKDS 1,5/3-5,08 power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, J3 Molex KK-254 22-27-2031 priva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, J4 TST040HDBC-42 panel, J8 Samtec TSW-108-07-G-S JTAG (b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, J9 Samtec TSW-104-07-G-S buttons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, Q1 SQJ460AEP (AEC-Q101, 60V/20V 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, Q2 SQJ460AEP (AEC-Q101, 60V/20V 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, Q3 PMV55ENEA ignition wake pulld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, U1 LM74930-Q1, U10 TLV767-Q1 (3.3 V audio AVDD), U11 TPS2557-Q1, U12 TPD4E02B04-Q1 line-out ESD (b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, U13 TPD4E05U06-Q1 mic ESD, U14 TPD4E05U06-Q1 USB ESD, U15 TPS22918-Q1 (AEC-Q100 G2) MFi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, U2 LM61460-Q1, U3 TLV767-Q1, U4 TCAN1044V-Q1, U6 TPS65131-Q1, U7 TPS61165-Q1, U8 TPS22918-Q1 (AEC-Q100 G2) dia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, U9 TAC5112-Q1

Commit message: Six layers with solid GND planes, a field-solved DSI geometry, and the RGB variant routed
Both boards and display-rgb/ move to JLC06161H-3313 six-layer: F / In1 GND /
In2 / In3 with the +5V or +3V3 pour / In4 GND / B. Every net class except GND
is restricted to F, In2, In3 and B in the router input (FreeRouting 2.2.4
ignores a layer_rule "active off"), and review/layout_checks.py now fails a
board with any track on In1 or In4. All three boards: 0 unconnected under
kicad-cli DRC, accepted categories only, no copper but GND fill on the planes.

- DSI pairs are 0.16 mm, field-solved on the new stack-up at 96.4-103.1 ohm
  differential (review/dsi_impedance.py); board minimum track 0.15 mm.
- gauges/ routes VIN_PROT, VIN_FUSED and +5V at 0.4 mm from the start; every
  power net now passes the 20 K current check, and nothing crosses the buck's
  switch node (P-07).
- Panel bias +5.98 V / -6.05 V, inside the ICNL9707's rating; fab/README.md
  gives a diode-test check of the panel's pin polarity before JP1/JP2.
- display-rgb/ brought up to date with display/ (standoffs, FETs, audio,
  USB-C, MFi header), RGB parts renumbered, routed; still not a fab candidate
  while its panel connector is a placeholder.
- FreeRouting runs end at routing: (postroute off) in the DSN, a job timeout
  as backstop; one in-place attempt, since retries of one DSN are identical.
- The OV/UV divider tops are pulled to the LM74930 SW pin.
- docs/electrical-review.md section 8b records the measured results; the
  display/ battery path on inner copper (D-02 residual) is still open.

Co-Authored-By: Claude Opus 5.5 <noreply@anthropic.com>
Parts:
- R38: value 562k VPOS top R1 (see docstring) -> 511k VPOS top R1 (see docstring)
- R40: value 536k VNEG top R3 (see docstring) -> 499k VNEG top R3 (see docstring)
