File: display-rgb/ClusterDisplayRGB.kicad_sch (KiCad schematic)
At the start: 133 parts, among them J1 Verdin iMX95 Hexa 8GB WB IT, J10 RTC coin cell, J11 Molex KK-254 22-27-2041, rota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, J12 Samtec TSW-103-07-G-S A55 con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, J13 Samtec TSW-105-07-G-S USB_1 O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, J14 PLACEHOLDER 50-pin FPC for th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, J2 Phoenix MKDS 1,5/3-5,08 power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, J3 Molex KK-254 22-27-2031 priva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, J4 TST040HDBC-42 panel, J8 Samtec TSW-108-07-G-S JTAG (b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, J9 Samtec TSW-104-07-G-S buttons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, Q1 PMV55ENEA (AEC-Q101, 60V/20V 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, Q2 PMV55ENEA (AEC-Q101, 60V/20V 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, Q3 PMV55ENEA ignition wake pulld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, U1 LM74930-Q1, U10 TLV733P-Q1 3.3V (AEC-Q100 G1), U2 LM61460-Q1, U3 TLV767-Q1, U4 TCAN1044V-Q1, U6 TPS65131-Q1, U7 TPS61165-Q1, U8 TPS22918-Q1 (AEC-Q100 G2) dia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, U9 DS90CF384AQ-Q1

Commit message: Six layers with solid GND planes, a field-solved DSI geometry, and the RGB variant routed
Both boards and display-rgb/ move to JLC06161H-3313 six-layer: F / In1 GND /
In2 / In3 with the +5V or +3V3 pour / In4 GND / B. Every net class except GND
is restricted to F, In2, In3 and B in the router input (FreeRouting 2.2.4
ignores a layer_rule "active off"), and review/layout_checks.py now fails a
board with any track on In1 or In4. All three boards: 0 unconnected under
kicad-cli DRC, accepted categories only, no copper but GND fill on the planes.

- DSI pairs are 0.16 mm, field-solved on the new stack-up at 96.4-103.1 ohm
  differential (review/dsi_impedance.py); board minimum track 0.15 mm.
- gauges/ routes VIN_PROT, VIN_FUSED and +5V at 0.4 mm from the start; every
  power net now passes the 20 K current check, and nothing crosses the buck's
  switch node (P-07).
- Panel bias +5.98 V / -6.05 V, inside the ICNL9707's rating; fab/README.md
  gives a diode-test check of the panel's pin polarity before JP1/JP2.
- display-rgb/ brought up to date with display/ (standoffs, FETs, audio,
  USB-C, MFi header), RGB parts renumbered, routed; still not a fab candidate
  while its panel connector is a placeholder.
- FreeRouting runs end at routing: (postroute off) in the DSN, a job timeout
  as backstop; one in-place attempt, since retries of one DSN are identical.
- The OV/UV divider tops are pulled to the LM74930 SW pin.
- docs/electrical-review.md section 8b records the measured results; the
  display/ battery path on inner copper (D-02 residual) is still open.

Co-Authored-By: Claude Opus 5.5 <noreply@anthropic.com>
Parts:
- removed C46: 22u VPOS out 16V (AEC-Q200), Capacitor_SMD:C_1206_3216Metric, symbol ClusterDisplayRGB:C_1206
- removed C47: 22u VNEG out 16V (AEC-Q200), Capacitor_SMD:C_1206_3216Metric, symbol ClusterDisplayRGB:C_1206
- removed C64: 1u LDO input (AEC-Q200), Capacitor_SMD:C_0603_1608Metric, symbol ClusterDisplayRGB:C
- removed C65: 1u LDO output (AEC-Q200), Capacitor_SMD:C_0603_1608Metric, symbol ClusterDisplayRGB:C
- removed C66, C68, C70: 100n receiver VCC decoupling (AEC-Q200), Capacitor_SMD:C_0603_1608Metric, symbol ClusterDisplayRGB:C
- removed C72: 10u receiver bulk (AEC-Q200), Capacitor_SMD:C_0805_2012Metric, symbol ClusterDisplayRGB:C_0805
- removed J14: PLACEHOLDER 50-pin FPC for the RGB panel (pinout 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, Connector_FFC-FPC:Hirose_FH12-50S-0.5SH_1x50-1MP_P0.50mm_Horizontal, symbol ClusterDisplayRGB:CONN_RGB
- removed Q1: PMV55ENEA (AEC-Q101, 60V/20V VGS) diode, Package_TO_SOT_SMD:SOT-23, symbol ClusterDisplayRGB:NFET
- removed Q2: PMV55ENEA (AEC-Q101, 60V/20V VGS) pass, Package_TO_SOT_SMD:SOT-23, symbol ClusterDisplayRGB:NFET
- removed U10: TLV733P-Q1 3.3V (AEC-Q100 G1), Package_TO_SOT_SMD:SOT-23-5, symbol ClusterDisplayRGB:TLV733P-Q1
- removed U9: DS90CF384AQ-Q1, Package_SO:TSSOP-56_6.1x14mm_P0.5mm, symbol ClusterDisplayRGB:DS90CF384AQ-Q1
- added C46: 22u VPOS out 16V (AEC-Q200), Capacitor_SMD:C_1210_3225Metric, symbol ClusterDisplayRGB:C_1210
- added C47: 22u VNEG out 16V (AEC-Q200), Capacitor_SMD:C_1210_3225Metric, symbol ClusterDisplayRGB:C_1210
- added C64: 10u CIN, Capacitor_SMD:C_0805_2012Metric, symbol ClusterDisplayRGB:C_0805
- added C65: 10u COUT, Capacitor_SMD:C_0805_2012Metric, symbol ClusterDisplayRGB:C_0805
- added C66: 10u AVDD, Capacitor_SMD:C_0805_2012Metric, symbol ClusterDisplayRGB:C_0805
- added C68: 10u DREG, Capacitor_SMD:C_0805_2012Metric, symbol ClusterDisplayRGB:C_0805
- added C70: 10u IOVDD, Capacitor_SMD:C_0805_2012Metric, symbol ClusterDisplayRGB:C_0805
- added C72: 1u VREF, Capacitor_SMD:C_0603_1608Metric, symbol ClusterDisplayRGB:C
- added C73: 1u MICBIAS, Capacitor_SMD:C_0603_1608Metric, symbol ClusterDisplayRGB:C
- added C74, C75: 1u mic AC couple, Capacitor_SMD:C_0603_1608Metric, symbol ClusterDisplayRGB:C
- added C76, C77, C78, C79: 4.7u line-out DC block, Capacitor_SMD:C_0805_2012Metric, symbol ClusterDisplayRGB:C_0805
- added C80: 100n USB switch IN, Capacitor_SMD:C_0603_1608Metric, symbol ClusterDisplayRGB:C
- added C81: 10u USB switch IN, Capacitor_SMD:C_0805_2012Metric, symbol ClusterDisplayRGB:C_0805
- added C82: 100u 35V hybrid polymer VBUS (Panasonic EEH-ZA1V1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, Capacitor_SMD:CP_Elec_8x10, symbol ClusterDisplayRGB:CP_HYBRID
- added C83: 1u MFi switch CIN, Capacitor_SMD:C_0603_1608Metric, symbol ClusterDisplayRGB:C
- added C84: 1u MFi 5V out, Capacitor_SMD:C_0603_1608Metric, symbol ClusterDisplayRGB:C
- added C85: 1u LDO input (AEC-Q200), Capacitor_SMD:C_0603_1608Metric, symbol ClusterDisplayRGB:C
- added C86: 1u LDO output (AEC-Q200), Capacitor_SMD:C_0603_1608Metric, symbol ClusterDisplayRGB:C
- added C87, C88, C89, C90, C91, C92: 100n receiver VCC decoupling (AEC-Q200), Capacitor_SMD:C_0603_1608Metric, symbol ClusterDisplayRGB:C
- added C93: 10u receiver bulk (AEC-Q200), Capacitor_SMD:C_0805_2012Metric, symbol ClusterDisplayRGB:C_0805
- added D8: SMAJ5.0A VBUS TVS, Diode_SMD:D_SMA, symbol ClusterDisplayRGB:TVS_SMA
- added J14: JST XH B5B-XH-A balanced line-out L/R, Connector_JST:JST_XH_B5B-XH-A_1x05_P2.50mm_Vertical, symbol ClusterDisplayRGB:CONN_LINEOUT
- added J15: JST XH B3B-XH-A electret microphone (2-wire + shi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, Connector_JST:JST_XH_B3B-XH-A_1x03_P2.50mm_Vertical, symbol ClusterDisplayRGB:CONN_MIC
- added J16: MFi daughterboard header I2C_1, reset, switched 5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, Connector_PinHeader_2.54mm:PinHeader_1x06_P2.54mm_Vertical, symbol ClusterDisplayRGB:CONN_MFI
- added J17: GCT USB4105-GF-A USB-C 2.0 host receptacle, Connector_USB:USB_C_Receptacle_GCT_USB4105-xx-A_16P_TopMnt_Horizontal, symbol ClusterDisplayRGB:CONN_USBC
- added J18: PLACEHOLDER 50-pin FPC for the RGB panel (pinout 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, Connector_FFC-FPC:Hirose_FH12-50S-0.5SH_1x50-1MP_P0.50mm_Horizontal, symbol ClusterDisplayRGB:CONN_RGB
- added Q1: SQJ460AEP (AEC-Q101, 60V/20V VGS) diode, Package_SO:PowerPAK_SO-8L_Single, symbol ClusterDisplayRGB:NFET_PWR
- added Q2: SQJ460AEP (AEC-Q101, 60V/20V VGS) pass, Package_SO:PowerPAK_SO-8L_Single, symbol ClusterDisplayRGB:NFET_PWR
- added R65, R66, R67, R68: 100R line-out series, Resistor_SMD:R_0603_1608Metric, symbol ClusterDisplayRGB:R
- added R69: 61.9k 1% USB ILIM (1.6-2.0 A), Resistor_SMD:R_0603_1608Metric, symbol ClusterDisplayRGB:R
- added R70: 100k FAULT pull-up to +1V8, Resistor_SMD:R_0603_1608Metric, symbol ClusterDisplayRGB:R
- added R71: 22k Rp CC1 (1.5 A, +/-5 percent or better), Resistor_SMD:R_0603_1608Metric, symbol ClusterDisplayRGB:R
- added R72: 22k Rp CC2 (1.5 A, +/-5 percent or better), Resistor_SMD:R_0603_1608Metric, symbol ClusterDisplayRGB:R
- added R73: 100k USB EN pull-down, Resistor_SMD:R_0603_1608Metric, symbol ClusterDisplayRGB:R
- added R74: 100k MFi switch off in reset, Resistor_SMD:R_0603_1608Metric, symbol ClusterDisplayRGB:R
- added R75, R76, R77, R78, R79: 100R LVDS pair termination, Resistor_SMD:R_0603_1608Metric, symbol ClusterDisplayRGB:R
- added R80: 10k PWR_DWN pull-up (always enabled), Resistor_SMD:R_0603_1608Metric, symbol ClusterDisplayRGB:R
- added U10: TLV767-Q1 (3.3 V audio AVDD), Package_DFN_QFN:Texas_DRB0008A, symbol ClusterDisplayRGB:TLV767-Q1
- added U11: TPS2557-Q1, Package_DFN_QFN:Texas_DRB0008A, symbol ClusterDisplayRGB:TPS2557-Q1
- added U12: TPD4E02B04-Q1 line-out ESD (bidirectional, review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, Package_SON:USON-10_2.5x1.0mm_P0.5mm, symbol ClusterDisplayRGB:TPD4E02B04-Q1
- added U13: TPD4E05U06-Q1 mic ESD, Package_SON:USON-10_2.5x1.0mm_P0.5mm, symbol ClusterDisplayRGB:TPD4E05U06-Q1
- added U14: TPD4E05U06-Q1 USB ESD, Package_SON:USON-10_2.5x1.0mm_P0.5mm, symbol ClusterDisplayRGB:TPD4E05U06-Q1
- added U15: TPS22918-Q1 (AEC-Q100 G2) MFi 5V switch, Package_TO_SOT_SMD:SOT-23-6, symbol ClusterDisplayRGB:TPS22918-Q1
- added U16: DS90CF384AQ-Q1, Package_SO:TSSOP-56_6.1x14mm_P0.5mm, symbol ClusterDisplayRGB:DS90CF384AQ-Q1
- added U17: TLV733P-Q1 3.3V (AEC-Q100 G1), Package_TO_SOT_SMD:SOT-23-5, symbol ClusterDisplayRGB:TLV733P-Q1
- added U9: TAC5112-Q1, Package_DFN_QFN:QFN-32-1EP_5x5mm_P0.5mm_EP3.7x3.7mm_ThermalVias, symbol ClusterDisplayRGB:TAC5112-Q1
- C67: value 100n receiver VCC decoupling (AEC-Q200) -> 100n AVDD
- C69: value 100n receiver VCC decoupling (AEC-Q200) -> 100n DREG
- C71: value 100n receiver VCC decoupling (AEC-Q200) -> 100n IOVDD
- D1: footprint Diode_SMD:D_SMB -> Diode_SMD:D_SMC
- R38: value 562k VPOS top R1 (see docstring) -> 511k VPOS top R1 (see docstring)
- R40: value 536k VNEG top R3 (see docstring) -> 499k VNEG top R3 (see docstring)
- R59: value 100R LVDS pair termination -> 316k 1% FB top
- R60: value 100R LVDS pair termination -> 100k FB bot
- R61: value 100R LVDS pair termination -> 2.2k I2C1 SDA pull-up
- R62: value 100R LVDS pair termination -> 2.2k I2C1 SCL pull-up
- R63: value 100R LVDS pair termination -> 2.2k mic bias
- R64: value 10k PWR_DWN pull-up (always enabled) -> 100R mic return
Connections:
- net +12V_PROT: now also Q1.5 (D)
- net +1V8: now also C71.1, R61.2, R62.2, C70.1, J16.6 (V1V8), J18.13 (V1V8), R70.2, U9.7 (IOVDD)
- net +3V3: now also R59.1, C65.1, C66.1, U10.1 (OUT), U9.31 (AVDD); no longer C69.1, C71.1, R64.1
- net +5V: now also C64.1, C80.1, C81.1, C83.1, C85.1, R71.2, R72.2, U10.8 (IN), U11.2 (IN1), U11.3 (IN2), U15.1 (VIN), U17.1 (IN), U17.3 (EN)
- net COMMON: now also Q1.1 (S1), Q1.2 (S2), Q1.3 (S3), Q2.1 (S1), Q2.2 (S2), Q2.3 (S3)
- net DGATE: now also Q1.4 (G)
- net GND: now also R60.2, R64.2, C46.2, C47.2, C64.2, C65.2, C66.2, C68.2, C70.2, C72.2, C73.2, C80.2, C81.2, C82.2, C83.2, C84.2, C85.2, C86.2, C87.2, C88.2, C89.2, C90.2, C91.2, C92.2, C93.2, D8.2, J14.5 (GND), J15.3 (GND), J16.4 (GND), J17.A1 (A1_GND), J17.A12 (A12_GND), J17.B1 (B1_GND), J17.B12 (B12_GND), J17.SH (SHIELD), J18.1 (GND1), J18.15 (GND3), J18.24 (GND4), J18.33 (GND5), J18.42 (GND6), J18.47 (GND7), J18.50 (GND8), J18.6 (GND2), R69.2, R73.2, R74.2, U10.4 (GND), U10.6 (GND2), U10.9 (EP), U11.1 (GND), U11.9 (EP), U12.3 (GND1), U12.8 (GND2), U13.3 (GND1), U13.8 (GND2), U14.3 (GND1), U14.8 (GND2), U15.2 (GND), U16.14 (LVDS_GND2), U16.21 (LVDS_GND3), U16.22 (PLL_GND1), U16.24 (PLL_GND2), U16.28 (GND2), U16.36 (GND3), U16.4 (GND1), U16.44 (GND4), U16.52 (GND5), U16.8 (LVDS_GND1), U17.2 (GND), U9.1 (VSS1), U9.15 (VSS3), U9.16 (ADDR), U9.22 (VSSI1), U9.23 (VSSI2), U9.24 (VSSI3), U9.25 (VSSI4), U9.26 (VSS4), U9.33 (EP), U9.8 (VSS2)
- net HGATE: now also Q2.4 (G)
- net LVDS_CLK_N: now also R79.2, U16.17 (RxCLKIN-); no longer R63.2
- net LVDS_CLK_P: now also R79.1, U16.18 (RxCLKIN+); no longer R63.1
- net LVDS_D0_N: now also R75.2, U16.9 (RxIN0-); no longer R59.2
- net LVDS_D0_P: now also R75.1, U16.10 (RxIN0+); no longer R59.1
- net LVDS_D1_N: now also R76.2, U16.11 (RxIN1-); no longer R60.2
- net LVDS_D1_P: now also R76.1, U16.12 (RxIN1+); no longer R60.1
- net LVDS_D2_N: now also J1.106 (LVDS0_D2_N), R77.2, U16.15 (RxIN2-); no longer J1.106 (LVDS0_D2_N), R61.2
- net LVDS_D2_P: now also R77.1, U16.16 (RxIN2+); no longer R61.1
- net LVDS_D3_N: now also R78.2, U16.19 (RxIN3-); no longer R62.2
- net LVDS_D3_P: now also R78.1, U16.20 (RxIN3+); no longer R62.1
- net PANEL_VSN: now also C47.1
- net PANEL_VSP: now also C46.1
- net PWR_EN_MOCI: now also U10.5 (EN)
- net RGB_B0: now also J18.16 (B0), U16.47 (RxOUT15)
- net RGB_B1: now also J18.17 (B1), U16.51 (RxOUT18)
- net RGB_B2: now also J18.18 (B2), U16.53 (RxOUT19)
- net RGB_B3: now also J18.19 (B3), U16.54 (RxOUT20)
- net RGB_B4: now also J18.20 (B4), U16.55 (RxOUT21)
- net RGB_B5: now also J18.21 (B5), U16.1 (RxOUT22)
- net RGB_B6: now also J18.22 (B6), U16.49 (RxOUT16)
- net RGB_B7: now also J18.23 (B7), U16.50 (RxOUT17)
- net RGB_DE: now also J18.46 (DE), U16.6 (RxOUT26)
- net RGB_G0: now also J18.25 (G0), U16.37 (RxOUT7)
- net RGB_G1: now also J18.26 (G1), U16.38 (RxOUT8)
- net RGB_G2: now also J18.27 (G2), U16.39 (RxOUT9)
- net RGB_G3: now also J18.28 (G3), U16.43 (RxOUT12)
- net RGB_G4: now also J18.29 (G4), U16.45 (RxOUT13)
- net RGB_G5: now also J18.30 (G5), U16.46 (RxOUT14)
- net RGB_G6: now also J18.31 (G6), U16.41 (RxOUT10)
- net RGB_G7: now also J18.32 (G7), U16.42 (RxOUT11)
- net RGB_HS: now also J18.44 (HS), U16.3 (RxOUT24)
- net RGB_LEDA: now also J18.4 (LEDA1), J18.5 (LEDA2)
- net RGB_LEDK: now also J18.2 (LEDK1), J18.3 (LEDK2)
- net RGB_PCLK: now also J18.43 (PCLK), U16.26 (RxCLK_OUT)
- net RGB_PWRDN: now also R80.2, U16.25 (PWR_DWN); no longer R64.2
- net RGB_R0: now also J18.34 (R0), U16.27 (RxOUT0)
- net RGB_R1: now also J18.35 (R1), U16.29 (RxOUT1)
- net RGB_R2: now also J18.36 (R2), U16.30 (RxOUT2)
- net RGB_R3: now also J18.37 (R3), U16.32 (RxOUT3)
- net RGB_R4: now also J18.38 (R4), U16.33 (RxOUT4)
- net RGB_R5: now also J18.39 (R5), U16.35 (RxOUT6)
- net RGB_R6: now also J18.40 (R6), U16.7 (RxOUT27)
- net RGB_R7: now also J18.41 (R7), U16.34 (RxOUT5)
- net RGB_RESET: now also J1.212 (GPIO_4), J18.7 (RESET); no longer J1.208 (GPIO_2)
- net RGB_SPI_CLK: now also J18.9 (SPI_CLK)
- net RGB_SPI_CS: now also J18.8 (SPI_CS)
- net RGB_SPI_SDA: now also J18.10 (SPI_SDA)
- net RGB_VS: now also J18.45 (VS), U16.5 (RxOUT25)
- net SENSE_OUT: now also Q2.5 (D)
- net MFI_PWR_EN: now reaches J1.210 (GPIO_3)
- net MFI_PWR_EN: now also R74.1, U15.3 (ON)
- new net +3V3_RGB: C86.1, C87.1, C88.1, C89.1, C90.1, C91.1, C92.1, C93.1, J18.11 (V3V31), J18.12 (V3V32), R80.1, U16.13 (LVDS_VCC), U16.23 (PLL_VCC), U16.31 (VCC1), U16.40 (VCC2), U16.48 (VCC3), U16.56 (VCC4), U17.5 (OUT)
- new net AOUT_L_N: R66.1, U9.27 (OUT1M)
- new net AOUT_L_N_R: C77.1, R66.2
- new net AOUT_L_P: R65.1, U9.28 (OUT1P)
- new net AOUT_L_P_R: C76.1, R65.2
- new net AOUT_R_N: R68.1, U9.30 (OUT2M)
- new net AOUT_R_N_R: C79.1, R68.2
- new net AOUT_R_P: R67.1, U9.29 (OUT2P)
- new net AOUT_R_P_R: C78.1, R67.2
- new net CODEC_DREG: C68.1, C69.1, U9.2 (DREG)
- new net CODEC_MICBIAS: C73.1, R63.1, U9.17 (MICBIAS)
- new net CODEC_VREF: C72.1, U9.32 (VREF)
- new net FB_3V3: R59.2, R60.1, U10.3 (FB)
- new net I2C1_SCL: J1.14 (I2C_1_SCL), J16.2 (SCL), R62.1, U9.9 (SCL)
- new net I2C1_SDA: J1.12 (I2C_1_SDA), J16.1 (SDA), R61.1, U9.10 (SDA)
- new net I2S_BCLK: J1.30 (I2S_1_BCLK), U9.3 (BCLK)
- new net I2S_DIN: J1.34 (I2S_1_D_OUT), U9.6 (DIN)
- new net I2S_DOUT: J1.36 (I2S_1_D_IN), U9.5 (DOUT)
- new net I2S_FSYNC: J1.32 (I2S_1_SYNC), U9.4 (FSYNC)
- new net LINE_L_N: C77.2, J14.2 (L_N), U12.2 (CH2)
- new net LINE_L_P: C76.2, J14.1 (L_P), U12.1 (CH1)
- new net LINE_R_N: C79.2, J14.4 (R_N), U12.5 (CH4)
- new net LINE_R_P: C78.2, J14.3 (R_P), U12.4 (CH3)
- new net MFI_5V: C84.1, J16.5 (VSW), U15.6 (VOUT)
- new net MFI_RST_N: J1.208 (GPIO_2), J16.3 (RST_N)
- new net MIC_IN_N: C75.2, U9.19 (IN1M)
- new net MIC_IN_P: C74.2, U9.18 (IN1P)
- new net MIC_N: C75.1, J15.2 (MIC_N), R64.1, U13.2 (CH2)
- new net MIC_P: C74.1, J15.1 (MIC_P), R63.2, U13.1 (CH1)
- new net USB2_CC1: J17.A5 (A5_CC1), R71.1, U14.4 (CH3)
- new net USB2_CC2: J17.B5 (B5_CC2), R72.1, U14.5 (CH4)
- new net USB2_DN: J1.181 (USB_2_D_N), J17.A7 (A7_DN), J17.B7 (B7_DN), U14.2 (CH2)
- new net USB2_DP: J1.183 (USB_2_D_P), J17.A6 (A6_DP), J17.B6 (B6_DP), U14.1 (CH1)
- new net USB2_EN: J1.185 (USB_2_EN), R73.1, U11.4 (EN)
- new net USB2_ILIM: R69.1, U11.5 (ILIM)
- new net USB2_OC_N: J1.187 (USB_2_OC#), R70.1, U11.8 (FAULT)
- new net USB2_VBUS: C82.1, D8.1, J17.A9 (A9_VBUS), J17.B4 (B4_VBUS), U11.6 (OUT1), U11.7 (OUT2)
- new net USB2_VBUS_L: J17.A4 (A4_VBUS), J17.B9 (B9_VBUS)
- no-connect marks 183 -> 197
